File: LeashPCB/LeashPCB.sch (KiCad schematic (older format))
At the start: 4 parts

Commit message: Started adding battery holder info (built ins)
Parts:
- added BT1: Reference Battery Holder, Battery:BatteryHolder_Keystone_2468_2xAAA, symbol Device:Battery
- added C1: C, symbol Device:C
- added J1: Conn_02x03_Odd_Even, symbol Connector_Generic:Conn_02x03_Odd_Even
- added SW1: SW_Push, symbol Switch:SW_Push
- added U?: 5204, symbol LeashPCB:5204
- added U?: 5212, symbol LeashPCB:5212
- added U?: 5226, symbol LeashPCB:5226
- U1: renamed from U?; footprint (none) -> Package_DFN_QFN:QFN-48-1EP_7x7mm_P0.5mm_EP5.15x5.15mm_ThermalVias
Connections:
- new net 3V3: C1.1, J1.1 (Pin_1)
- new net 3V_in: U?.1 (Pos)
- new net GND: C1.2, J1.5 (Pin_5), U?.1 (Neg)
- new net TCK: J1.4 (Pin_4)
- new net TDO: J1.6 (Pin_6)
- new net TMS: J1.2 (Pin_2)
- new net ~RESET: J1.3 (Pin_3)
