File: hw/LeashPCB/Indicators.sch (KiCad schematic (older format))
At the start: 0 parts

Commit message: Added more top level signals to block diagram and added alternate population options for power
Parts:
- added D? (x6): LED, symbol Device:LED
- added R? (x6): R, symbol Device:R
Connections:
- net labels added: 2.4G, 900MHz, Click1, Click2, GND, Power, User
- wire segments 0 -> 24

Commit message: Shifted all components to the left on the layout and added passives
Parts:
- D701, D702, D703, D704, D705, D706: renamed from D?; footprint (none) -> LED_SMD:LED_0402_1005Metric
- R701, R702, R703, R704, R705, R706: renamed from R?; footprint (none) -> Resistor_SMD:R_0402_1005Metric
Changed lines of the file:
@@
 Click2
 $Comp
-L Device:LED D?
+L Device:LED D701
 U 1 1 5D1F28D2
 P 4300 3625
-F 0 "D?" V 4339 3508 50  0000 R CNN
+F 0 "D701" V 4339 3508 50  0000 R CNN
 F 1 "LED" V 4248 3508 50  0000 R CNN
-F 2 "" H 4300 3625 50  0001 C CNN
+F 2 "LED_SMD:LED_0402_1005Metric" H 4300 3625 50  0001 C CNN
 F 3 "~" H 4300 3625 50  0001 C CNN
 	1    4300 3625
@@
 $EndComp
 $Comp
-L Device:R R?
+L Device:R R701
 U 1 1 5D1F2C92
 P 4300 4100
-F 0 "R?" H 4370 4146 50  0000 L CNN
+F 0 "R701" H 4370 4146 50  0000 L CNN
 F 1 "R" H 4370 4055 50  0000 L CNN
-F 2 "" V 4230 4100 50  0001 C CNN
+F 2 "Resistor_SMD:R_0402_1005Metric" V 4230 4100 50  0001 C CNN
 F 3 "~" H 4300 4100 50  0001 C CNN
 	1    4300 4100
@@
 	4300 4250 4300 4475
 $Comp
-L power:GND #PWR?
+L power:GND #PWR0108
 U 1 1 5D1F308C
 P 4300 4475
-F 0 "#PWR?" H 4300 4225 50  0001 C CNN
+F 0 "#PWR0108" H 4300 4225 50  0001 C CNN
 F 1 "GND" H 4305 4302 50  0000 C CNN
 F 2 "" H 4300 4475 50  0001 C CNN
@@
 $EndComp
 $Comp
-L Device:LED D?
+L Device:LED D702
 U 1 1 5D1F3B0B
 P 4750 3625
-F 0 "D?" V 4789 3508 50  0000 R CNN
+F 0 "D702" V 4789 3508 50  0000 R CNN
 F 1 "LED" V 4698 3508 50  0000 R CNN
-F 2 "" H 4750 3625 50  0001 C CNN
+F 2 "LED_SMD:LED_0402_1005Metric" H 4750 3625 50  0001 C CNN
 F 3 "~" H 4750 3625 50  0001 C CNN
 	1    4750 3625
@@
 $EndComp
 $Comp
-L Device:R R?
+L Device:R R702
 U 1 1 5D1F3B15
 P 4750 4100
-F 0 "R?" H 4820 4146 50  0000 L CNN
+F 0 "R702" H 4820 4146 50  0000 L CNN
 F 1 "R" H 4820 4055 50  0000 L CNN
-F 2 "" V 4680 4100 50  0001 C CNN
+F 2 "Resistor_SMD:R_0402_1005Metric" V 4680 4100 50  0001 C CNN
 F 3 "~" H 4750 4100 50  0001 C CNN
 	1    4750 4100
@@
 	4750 4250 4750 4475
 $Comp
-L power:GND #PWR?
+L power:GND #PWR0109
 U 1 1 5D1F3B22
 P 4750 4475
-F 0 "#PWR?" H 4750 4225 50  0001 C CNN
+F 0 "#PWR0109" H 4750 4225 50  0001 C CNN
 F 1 "GND" H 4755 4302 50  0000 C CNN
 F 2 "" H 4750 4475 50  0001 C CNN
@@
 $EndComp
 $Comp
-L Device:LED D?
+L Device:LED D703
 U 1 1 5D1F5389
 P 5150 3625
-F 0 "D?" V 5189 3508 50  0000 R CNN
+F 0 "D703" V 5189 3508 50  0000 R CNN
 F 1 "LED" V 5098 3508 50  0000 R CNN
-F 2 "" H 5150 3625 50  0001 C CNN
+F 2 "LED_SMD:LED_0402_1005Metric" H 5150 3625 50  0001 C CNN
 F 3 "~" H 5150 3625 50  0001 C CNN
 	1    5150 3625
@@
 $EndComp
 $Comp
-L Device:R R?
+L Device:R R703
 U 1 1 5D1F5393
 P 5150 4100
-F 0 "R?" H 5220 4146 50  0000 L CNN
+F 0 "R703" H 5220 4146 50  0000 L CNN
 F 1 "R" H 5220 4055 50  0000 L CNN
-F 2 "" V 5080 4100 50  0001 C CNN
+F 2 "Resistor_SMD:R_0402_1005Metric" V 5080 4100 50  0001 C CNN
 F 3 "~" H 5150 4100 50  0001 C CNN
 	1    5150 4100
@@
 	5150 4250 5150 4475
 $Comp
-L power:GND #PWR?
+L power:GND #PWR0110
 U 1 1 5D1F53A0
 P 5150 4475
-F 0 "#PWR?" H 5150 4225 50  0001 C CNN
+F 0 "#PWR0110" H 5150 4225 50  0001 C CNN
 F 1 "GND" H 5155 4302 50  0000 C CNN
 F 2 "" H 5150 4475 50  0001 C CNN
@@
 $EndComp
 $Comp
-L Device:LED D?
+L Device:LED D704
 U 1 1 5D1F53AA
 P 5600 3625
-F 0 "D?" V 5639 3508 50  0000 R CNN
+F 0 "D704" V 5639 3508 50  0000 R CNN
 F 1 "LED" V 5548 3508 50  0000 R CNN
-F 2 "" H 5600 3625 50  0001 C CNN
+F 2 "LED_SMD:LED_0402_1005Metric" H 5600 3625 50  0001 C CNN
 F 3 "~" H 5600 3625 50  0001 C CNN
 	1    5600 3625
@@
 $EndComp
 $Comp
-L Device:R R?
+L Device:R R704
 U 1 1 5D1F53B4
 P 5600 4100
-F 0 "R?" H 5670 4146 50  0000 L CNN
+F 0 "R704" H 5670 4146 50  0000 L CNN
 F 1 "R" H 5670 4055 50  0000 L CNN
-F 2 "" V 5530 4100 50  0001 C CNN
+F 2 "Resistor_SMD:R_0402_1005Metric" V 5530 4100 50  0001 C CNN
 F 3 "~" H 5600 4100 50  0001 C CNN
 	1    5600 4100
@@
 	5600 4250 5600 4475
 $Comp
-L power:GND #PWR?
+L power:GND #PWR0111
 U 1 1 5D1F53C1
 P 5600 4475
-F 0 "#PWR?" H 5600 4225 50  0001 C CNN
+F 0 "#PWR0111" H 5600 4225 50  0001 C CNN
 F 1 "GND" H 5605 4302 50  0000 C CNN
 F 2 "" H 5600 4475 50  0001 C CNN
@@
 $EndComp
 $Comp
-L Device:LED D?
+L Device:LED D705
 U 1 1 5D1F7859
 P 6025 3625
-F 0 "D?" V 6064 3508 50  0000 R CNN
+F 0 "D705" V 6064 3508 50  0000 R CNN
 F 1 "LED" V 5973 3508 50  0000 R CNN
-F 2 "" H 6025 3625 50  0001 C CNN
+F 2 "LED_SMD:LED_0402_1005Metric" H 6025 3625 50  0001 C CNN
 F 3 "~" H 6025 3625 50  0001 C CNN
 	1    6025 3625
@@
 $EndComp
 $Comp
-L Device:R R?
+L Device:R R705
 U 1 1 5D1F7863
 P 6025 4100
-F 0 "R?" H 6095 4146 50  0000 L CNN
+F 0 "R705" H 6095 4146 50  0000 L CNN
 F 1 "R" H 6095 4055 50  0000 L CNN
-F 2 "" V 5955 4100 50  0001 C CNN
+F 2 "Resistor_SMD:R_0402_1005Metric" V 5955 4100 50  0001 C CNN
 F 3 "~" H 6025 4100 50  0001 C CNN
 	1    6025 4100
@@
 	6025 4250 6025 4475
 $Comp
-L power:GND #PWR?
+L power:GND #PWR0112
 U 1 1 5D1F7870
 P 6025 4475
-F 0 "#PWR?" H 6025 4225 50  0001 C CNN
+F 0 "#PWR0112" H 6025 4225 50  0001 C CNN
 F 1 "GND" H 6030 4302 50  0000 C CNN
 F 2 "" H 6025 4475 50  0001 C CNN
@@
 $EndComp
 $Comp
-L Device:LED D?
+L Device:LED D706
 U 1 1 5D1F787A
 P 6475 3625
-F 0 "D?" V 6514 3508 50  0000 R CNN
+F 0 "D706" V 6514 3508 50  0000 R CNN
 F 1 "LED" V 6423 3508 50  0000 R CNN
-F 2 "" H 6475 3625 50  0001 C CNN
+F 2 "LED_SMD:LED_0402_1005Metric" H 6475 3625 50  0001 C CNN
 F 3 "~" H 6475 3625 50  0001 C CNN
 	1    6475 3625
@@
 $EndComp
 $Comp
-L Device:R R?
+L Device:R R706
 U 1 1 5D1F7884
 P 6475 4100
-F 0 "R?" H 6545 4146 50  0000 L CNN
+F 0 "R706" H 6545 4146 50  0000 L CNN
 F 1 "R" H 6545 4055 50  0000 L CNN
-F 2 "" V 6405 4100 50  0001 C CNN
+F 2 "Resistor_SMD:R_0402_1005Metric" V 6405 4100 50  0001 C CNN
 F 3 "~" H 6475 4100 50  0001 C CNN
 	1    6475 4100
@@
 	6475 4250 6475 4475
 $Comp
-L power:GND #PWR?
+L power:GND #PWR0113
 U 1 1 5D1F7891
 P 6475 4475
-F 0 "#PWR?" H 6475 4225 50  0001 C CNN
+F 0 "#PWR0113" H 6475 4225 50  0001 C CNN
 F 1 "GND" H 6480 4302 50  0000 C CNN
 F 2 "" H 6475 4475 50  0001 C CNN

Commit message: Resized schematic sheets for printing and remapped signals for matching Launchpad headers
Parts:
- removed D703: LED, LED_SMD:LED_0402_1005Metric, symbol Device:LED
- removed R703: R, Resistor_SMD:R_0402_1005Metric, symbol Device:R
Connections:
- net labels removed: User
- wire segments 24 -> 20
Other:
- moved on the sheet: R701, R702, R704, R705, R706
