File: hw/LeashPCB/Indicators.sch (KiCad schematic (older format))
At the start: 10 parts

Commit message: Added SWD connector on the back side as a backup for testing and continued routing
Other:
- moved on the sheet: R701, R702
Changed lines of the file:
@@
 L Device:LED D701
 U 1 1 5D1F28D2
-P 8550 5050
-F 0 "D701" V 8589 4933 50  0000 R CNN
-F 1 "LED" V 8498 4933 50  0000 R CNN
-F 2 "LED_SMD:LED_0402_1005Metric" H 8550 5050 50  0001 C CNN
-F 3 "~" H 8550 5050 50  0001 C CNN
-	1    8550 5050
-	0    -1   -1   0
-$EndComp
-$Comp
-L Device:R R701
-U 1 1 5D1F2C92
-P 8550 5525
-F 0 "R701" H 8620 5571 50  0000 L CNN
-F 1 "R" H 8620 5480 50  0000 L CNN
-F 2 "Resistor_SMD:R_0402_1005Metric" V 8480 5525 50  0001 C CNN
-F 3 "~" H 8550 5525 50  0001 C CNN
-	1    8550 5525
-	1    0    0    -1
-$EndComp
-Wire Wire Line
-	8550 5200 8550 5375
-Wire Wire Line
-	8550 5675 8550 5900
-$Comp
-L power:GND #PWR0108
-U 1 1 5D1F308C
-P 8550 5900
-F 0 "#PWR0108" H 8550 5650 50  0001 C CNN
-F 1 "GND" H 8555 5727 50  0000 C CNN
-F 2 "" H 8550 5900 50  0001 C CNN
-F 3 "" H 8550 5900 50  0001 C CNN
-	1    8550 5900
-	1    0    0    -1
-$EndComp
-$Comp
-L Device:LED D702
-U 1 1 5D1F3B0B
 P 9000 5050
-F 0 "D702" V 9039 4933 50  0000 R CNN
+F 0 "D701" V 9039 4933 50  0000 R CNN
 F 1 "LED" V 8948 4933 50  0000 R CNN
 F 2 "LED_SMD:LED_0402_1005Metric" H 9000 5050 50  0001 C CNN
@@
 $EndComp
 $Comp
-L Device:R R702
-U 1 1 5D1F3B15
+L Device:R R701
+U 1 1 5D1F2C92
 P 9000 5525
-F 0 "R702" H 9070 5571 50  0000 L CNN
+F 0 "R701" H 9070 5571 50  0000 L CNN
 F 1 "R" H 9070 5480 50  0000 L CNN
 F 2 "Resistor_SMD:R_0402_1005Metric" V 8930 5525 50  0001 C CNN
@@
 	9000 5675 9000 5900
 $Comp
-L power:GND #PWR0109
-U 1 1 5D1F3B22
+L power:GND #PWR0108
+U 1 1 5D1F308C
 P 9000 5900
-F 0 "#PWR0109" H 9000 5650 50  0001 C CNN
+F 0 "#PWR0108" H 9000 5650 50  0001 C CNN
 F 1 "GND" H 9005 5727 50  0000 C CNN
 F 2 "" H 9000 5900 50  0001 C CNN
@@
 	7100 4625 8550 4625
 Wire Wire Line
+	9000 4300 9000 4900
+Wire Wire Line
+	7100 4300 9000 4300
+Wire Wire Line
+	7100 3675 9850 3675
+Wire Wire Line
+	9850 3675 9850 4900
+Wire Wire Line
+	7100 3375 10275 3375
+Wire Wire Line
+	10275 3375 10275 4900
+Wire Wire Line
+	7100 3075 10725 3075
+Wire Wire Line
+	10725 3075 10725 4900
+Wire Wire Line
 	8550 4625 8550 4900
-Wire Wire Line
-	7100 4300 9000 4300
-Wire Wire Line
-	9000 4300 9000 4900
-Wire Wire Line
-	7100 3675 9850 3675
-Wire Wire Line
-	9850 3675 9850 4900
-Wire Wire Line
-	7100 3375 10275 3375
-Wire Wire Line
-	10275 3375 10275 4900
-Wire Wire Line
-	7100 3075 10725 3075
-Wire Wire Line
-	10725 3075 10725 4900
+$Comp
+L power:GND #PWR0109
+U 1 1 5D1F3B22
+P 8550 5900
+F 0 "#PWR0109" H 8550 5650 50  0001 C CNN
+F 1 "GND" H 8555 5727 50  0000 C CNN
+F 2 "" H 8550 5900 50  0001 C CNN
+F 3 "" H 8550 5900 50  0001 C CNN
+	1    8550 5900
+	1    0    0    -1
+$EndComp
+Wire Wire Line
+	8550 5675 8550 5900
+Wire Wire Line
+	8550 5200 8550 5375
+$Comp
+L Device:R R702
+U 1 1 5D1F3B15
+P 8550 5525
+F 0 "R702" H 8620 5571 50  0000 L CNN
+F 1 "R" H 8620 5480 50  0000 L CNN
+F 2 "Resistor_SMD:R_0402_1005Metric" V 8480 5525 50  0001 C CNN
+F 3 "~" H 8550 5525 50  0001 C CNN
+	1    8550 5525
+	1    0    0    -1
+$EndComp
+$Comp
+L Device:LED D702
+U 1 1 5D1F3B0B
+P 8550 5050
+F 0 "D702" V 8589 4933 50  0000 R CNN
+F 1 "LED" V 8498 4933 50  0000 R CNN
+F 2 "LED_SMD:LED_0402_1005Metric" H 8550 5050 50  0001 C CNN
+F 3 "~" H 8550 5050 50  0001 C CNN
+	1    8550 5050
+	0    -1   -1   0
+$EndComp
 $EndSCHEMATC

Commit message: Adding part info for ordering components
Parts:
- D701, D702, D704, D705, D706: Description (none) -> LED RED DIFFUSED 1608 SMD; Link1 (none) -> https://www.digikey.com/product-detail/en/rohm-semiconducto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; MPN1 (none) -> SML-D12U1WT86; Standard Price (none) -> $0.03565; Vendor1 (none) -> Rohm Semiconductor
Changed lines of the file:
@@
 F 2 "LED_SMD:LED_0402_1005Metric" H 9000 5050 50  0001 C CNN
 F 3 "~" H 9000 5050 50  0001 C CNN
+F 4 "LED RED DIFFUSED 1608 SMD" H 9000 5050 50  0001 C CNN "Description"
+F 5 "https://www.digikey.com/product-detail/en/rohm-semiconductor/SML-D12U1WT86/SML-D12U1WT86TR-ND/5843853" H 9000 5050 50  0001 C CNN "Link1"
+F 6 "SML-D12U1WT86" H 9000 5050 50  0001 C CNN "MPN1"
+F 7 "$0.03565" H 9000 5050 50  0001 C CNN "Standard Price"
+F 8 "Rohm Semiconductor" H 9000 5050 50  0001 C CNN "Vendor1"
 	1    9000 5050
 	0    -1   -1   0
@@
 F 2 "LED_SMD:LED_0402_1005Metric" H 9850 5050 50  0001 C CNN
 F 3 "~" H 9850 5050 50  0001 C CNN
+F 4 "LED RED DIFFUSED 1608 SMD" H 9850 5050 50  0001 C CNN "Description"
+F 5 "https://www.digikey.com/product-detail/en/rohm-semiconductor/SML-D12U1WT86/SML-D12U1WT86TR-ND/5843853" H 9850 5050 50  0001 C CNN "Link1"
+F 6 "SML-D12U1WT86" H 9850 5050 50  0001 C CNN "MPN1"
+F 7 "$0.03565" H 9850 5050 50  0001 C CNN "Standard Price"
+F 8 "Rohm Semiconductor" H 9850 5050 50  0001 C CNN "Vendor1"
 	1    9850 5050
 	0    -1   -1   0
@@
 F 2 "LED_SMD:LED_0402_1005Metric" H 10275 5050 50  0001 C CNN
 F 3 "~" H 10275 5050 50  0001 C CNN
+F 4 "LED RED DIFFUSED 1608 SMD" H 10275 5050 50  0001 C CNN "Description"
+F 5 "https://www.digikey.com/product-detail/en/rohm-semiconductor/SML-D12U1WT86/SML-D12U1WT86TR-ND/5843853" H 10275 5050 50  0001 C CNN "Link1"
+F 6 "SML-D12U1WT86" H 10275 5050 50  0001 C CNN "MPN1"
+F 7 "$0.03565" H 10275 5050 50  0001 C CNN "Standard Price"
+F 8 "Rohm Semiconductor" H 10275 5050 50  0001 C CNN "Vendor1"
 	1    10275 5050
 	0    -1   -1   0
@@
 F 2 "LED_SMD:LED_0402_1005Metric" H 10725 5050 50  0001 C CNN
 F 3 "~" H 10725 5050 50  0001 C CNN
+F 4 "LED RED DIFFUSED 1608 SMD" H 10725 5050 50  0001 C CNN "Description"
+F 5 "https://www.digikey.com/product-detail/en/rohm-semiconductor/SML-D12U1WT86/SML-D12U1WT86TR-ND/5843853" H 10725 5050 50  0001 C CNN "Link1"
+F 6 "SML-D12U1WT86" H 10725 5050 50  0001 C CNN "MPN1"
+F 7 "$0.03565" H 10725 5050 50  0001 C CNN "Standard Price"
+F 8 "Rohm Semiconductor" H 10725 5050 50  0001 C CNN "Vendor1"
 	1    10725 5050
 	0    -1   -1   0
@@
 F 2 "LED_SMD:LED_0402_1005Metric" H 8550 5050 50  0001 C CNN
 F 3 "~" H 8550 5050 50  0001 C CNN
+F 4 "LED RED DIFFUSED 1608 SMD" H 8550 5050 50  0001 C CNN "Description"
+F 5 "https://www.digikey.com/product-detail/en/rohm-semiconductor/SML-D12U1WT86/SML-D12U1WT86TR-ND/5843853" H 8550 5050 50  0001 C CNN "Link1"
+F 6 "SML-D12U1WT86" H 8550 5050 50  0001 C CNN "MPN1"
+F 7 "$0.03565" H 8550 5050 50  0001 C CNN "Standard Price"
+F 8 "Rohm Semiconductor" H 8550 5050 50  0001 C CNN "Vendor1"
 	1    8550 5050
 	0    -1   -1   0

Commit message: Finished added components and generated BOM for ordering all parts
Parts:
- D701, D702, D704, D705, D706: Short Description (none) -> LED RED DIFFUSED 1608 SMD
- R701, R702, R704, R705, R706: value R -> 1K; Description (none) -> RES SMD 1K OHM 5% 1/16W 0402; Link1 (none) -> https://www.digikey.com/product-detail/en/yageo/RC0402JR-07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; MPN1 (none) -> RC0402JR-071KL; Short Description (none) -> RES SMD 1K OHM 5% 1/16W 0402; Standard Price (none) -> $0.00139; Vendor1 (none) -> Yageo
Changed lines of the file:
@@
 Sheet 5 10
 Title "BeagleDust Leash PCB"
-Date "2019-07-22"
-Rev "1"
+Date "2019-08-12"
+Rev "A"
 Comp "Beagleboard.org"
 Comment1 "Schematic designed by Analog Life, LLC"
@@
 F 7 "$0.03565" H 9000 5050 50  0001 C CNN "Standard Price"
 F 8 "Rohm Semiconductor" H 9000 5050 50  0001 C CNN "Vendor1"
+F 9 "LED RED DIFFUSED 1608 SMD" H 9000 5050 50  0001 C CNN "Short Description"
 	1    9000 5050
 	0    -1   -1   0
@@
 P 9000 5525
 F 0 "R701" H 9070 5571 50  0000 L CNN
-F 1 "R" H 9070 5480 50  0000 L CNN
+F 1 "1K" H 9070 5480 50  0000 L CNN
 F 2 "Resistor_SMD:R_0402_1005Metric" V 8930 5525 50  0001 C CNN
 F 3 "~" H 9000 5525 50  0001 C CNN
+F 4 "RES SMD 1K OHM 5% 1/16W 0402" H 9000 5525 50  0001 C CNN "Description"
+F 5 "https://www.digikey.com/product-detail/en/yageo/RC0402JR-071KL/311-1.0KJRCT-ND/729355" H 9000 5525 50  0001 C CNN "Link1"
+F 6 "RC0402JR-071KL" H 9000 5525 50  0001 C CNN "MPN1"
+F 7 "$0.00139" H 9000 5525 50  0001 C CNN "Standard Price"
+F 8 "Yageo" H 9000 5525 50  0001 C CNN "Vendor1"
+F 9 "RES SMD 1K OHM 5% 1/16W 0402" H 9000 5525 50  0001 C CNN "Short Description"
 	1    9000 5525
 	1    0    0    -1
@@
 F 7 "$0.03565" H 9850 5050 50  0001 C CNN "Standard Price"
 F 8 "Rohm Semiconductor" H 9850 5050 50  0001 C CNN "Vendor1"
+F 9 "LED RED DIFFUSED 1608 SMD" H 9850 5050 50  0001 C CNN "Short Description"
 	1    9850 5050
 	0    -1   -1   0
@@
 P 9850 5525
 F 0 "R704" H 9920 5571 50  0000 L CNN
-F 1 "R" H 9920 5480 50  0000 L CNN
+F 1 "1K" H 9920 5480 50  0000 L CNN
 F 2 "Resistor_SMD:R_0402_1005Metric" V 9780 5525 50  0001 C CNN
 F 3 "~" H 9850 5525 50  0001 C CNN
+F 4 "RES SMD 1K OHM 5% 1/16W 0402" H 9850 5525 50  0001 C CNN "Description"
+F 5 "https://www.digikey.com/product-detail/en/yageo/RC0402JR-071KL/311-1.0KJRCT-ND/729355" H 9850 5525 50  0001 C CNN "Link1"
+F 6 "RC0402JR-071KL" H 9850 5525 50  0001 C CNN "MPN1"
+F 7 "$0.00139" H 9850 5525 50  0001 C CNN "Standard Price"
+F 8 "Yageo" H 9850 5525 50  0001 C CNN "Vendor1"
+F 9 "RES SMD 1K OHM 5% 1/16W 0402" H 9850 5525 50  0001 C CNN "Short Description"
 	1    9850 5525
 	1    0    0    -1
@@
 F 7 "$0.03565" H 10275 5050 50  0001 C CNN "Standard Price"
 F 8 "Rohm Semiconductor" H 10275 5050 50  0001 C CNN "Vendor1"
+F 9 "LED RED DIFFUSED 1608 SMD" H 10275 5050 50  0001 C CNN "Short Description"
 	1    10275 5050
 	0    -1   -1   0
@@
 P 10275 5525
 F 0 "R705" H 10345 5571 50  0000 L CNN
-F 1 "R" H 10345 5480 50  0000 L CNN
+F 1 "1K" H 10345 5480 50  0000 L CNN
 F 2 "Resistor_SMD:R_0402_1005Metric" V 10205 5525 50  0001 C CNN
 F 3 "~" H 10275 5525 50  0001 C CNN
+F 4 "RES SMD 1K OHM 5% 1/16W 0402" H 10275 5525 50  0001 C CNN "Description"
+F 5 "https://www.digikey.com/product-detail/en/yageo/RC0402JR-071KL/311-1.0KJRCT-ND/729355" H 10275 5525 50  0001 C CNN "Link1"
+F 6 "RC0402JR-071KL" H 10275 5525 50  0001 C CNN "MPN1"
+F 7 "$0.00139" H 10275 5525 50  0001 C CNN "Standard Price"
+F 8 "Yageo" H 10275 5525 50  0001 C CNN "Vendor1"
+F 9 "RES SMD 1K OHM 5% 1/16W 0402" H 10275 5525 50  0001 C CNN "Short Description"
 	1    10275 5525
 	1    0    0    -1
@@
 F 7 "$0.03565" H 10725 5050 50  0001 C CNN "Standard Price"
 F 8 "Rohm Semiconductor" H 10725 5050 50  0001 C CNN "Vendor1"
+F 9 "LED RED DIFFUSED 1608 SMD" H 10725 5050 50  0001 C CNN "Short Description"
 	1    10725 5050
 	0    -1   -1   0
@@
 P 10725 5525
 F 0 "R706" H 10795 5571 50  0000 L CNN
-F 1 "R" H 10795 5480 50  0000 L CNN
+F 1 "1K" H 10795 5480 50  0000 L CNN
 F 2 "Resistor_SMD:R_0402_1005Metric" V 10655 5525 50  0001 C CNN
 F 3 "~" H 10725 5525 50  0001 C CNN
+F 4 "RES SMD 1K OHM 5% 1/16W 0402" H 10725 5525 50  0001 C CNN "Description"
+F 5 "https://www.digikey.com/product-detail/en/yageo/RC0402JR-071KL/311-1.0KJRCT-ND/729355" H 10725 5525 50  0001 C CNN "Link1"
+F 6 "RC0402JR-071KL" H 10725 5525 50  0001 C CNN "MPN1"
+F 7 "$0.00139" H 10725 5525 50  0001 C CNN "Standard Price"
+F 8 "Yageo" H 10725 5525 50  0001 C CNN "Vendor1"
+F 9 "RES SMD 1K OHM 5% 1/16W 0402" H 10725 5525 50  0001 C CNN "Short Description"
 	1    10725 5525
 	1    0    0    -1
@@
 P 8550 5525
 F 0 "R702" H 8620 5571 50  0000 L CNN
-F 1 "R" H 8620 5480 50  0000 L CNN
+F 1 "1K" H 8620 5480 50  0000 L CNN
 F 2 "Resistor_SMD:R_0402_1005Metric" V 8480 5525 50  0001 C CNN
 F 3 "~" H 8550 5525 50  0001 C CNN
+F 4 "RES SMD 1K OHM 5% 1/16W 0402" H 8550 5525 50  0001 C CNN "Description"
+F 5 "https://www.digikey.com/product-detail/en/yageo/RC0402JR-071KL/311-1.0KJRCT-ND/729355" H 8550 5525 50  0001 C CNN "Link1"
+F 6 "RC0402JR-071KL" H 8550 5525 50  0001 C CNN "MPN1"
+F 7 "$0.00139" H 8550 5525 50  0001 C CNN "Standard Price"
+F 8 "Yageo" H 8550 5525 50  0001 C CNN "Vendor1"
+F 9 "RES SMD 1K OHM 5% 1/16W 0402" H 8550 5525 50  0001 C CNN "Short Description"
 	1    8550 5525
 	1    0    0    -1
@@
 F 7 "$0.03565" H 8550 5050 50  0001 C CNN "Standard Price"
 F 8 "Rohm Semiconductor" H 8550 5050 50  0001 C CNN "Vendor1"
+F 9 "LED RED DIFFUSED 1608 SMD" H 8550 5050 50  0001 C CNN "Short Description"
 	1    8550 5050
 	0    -1   -1   0

Commit message: Done with 90% of routing, but going to move the USB to serial and power chips to open up the pathways underneath the CC1352R
Connections:
- net labels added: LED1, LED2
- net labels removed: Click1, Click2
Changed lines of the file:
@@
 Power
 Text HLabel 7100 4300 0    98   Input ~ 0
-Click1
+LED1
 Text HLabel 7100 4625 0    98   Input ~ 0
-Click2
+LED2
 $Comp
 L Device:LED D701

Commit message: Migrated all hierarchical labels to global labels
Connections:
- net labels added: 3V3, 900M
- net labels removed: 900MHz, Power
Changed lines of the file:
@@
 Comment4 ""
 $EndDescr
-Text HLabel 7100 3075 0    98   Input ~ 0
-2.4G
-Text HLabel 7100 3375 0    98   Input ~ 0
-900MHz
-Text HLabel 7100 3675 0    98   Input ~ 0
-Power
-Text HLabel 7100 4300 0    98   Input ~ 0
-LED1
-Text HLabel 7100 4625 0    98   Input ~ 0
-LED2
 $Comp
 L Device:LED D701
@@
 	10275 3375 10275 4900
 Wire Wire Line
-	7100 3075 10725 3075
-Wire Wire Line
 	10725 3075 10725 4900
 Wire Wire Line
@@
 	0    -1   -1   0
 $EndComp
+Text GLabel 7075 3075 0    63   Input ~ 0
+2.4G
+Text GLabel 7100 3375 0    63   Input ~ 0
+900M
+Text GLabel 7100 3675 0    63   Input ~ 0
+3V3
+Text GLabel 7100 4300 0    63   Input ~ 0
+LED1
+Text GLabel 7100 4625 0    63   Input ~ 0
+LED2
+Wire Wire Line
+	7075 3075 10725 3075
 $EndSCHEMATC

Commit message: Removed two extra pullup resistors
Parts:
- renumbered D702 to D401, D701 to D402, D704 to D403, D705 to D404, D706 to D405, R702 to R401, R701 to R402, R704 to R403, R705 to R404, R706 to R405
Changed lines of the file:
@@
 $EndDescr
 $Comp
-L Device:LED D701
+L Device:LED D402
 U 1 1 5D1F28D2
 P 9000 5050
-F 0 "D701" V 9039 4933 50  0000 R CNN
+F 0 "D402" V 9039 4933 50  0000 R CNN
 F 1 "LED" V 8948 4933 50  0000 R CNN
 F 2 "LED_SMD:LED_0402_1005Metric" H 9000 5050 50  0001 C CNN
@@
 $EndComp
 $Comp
-L Device:R R701
+L Device:R R402
 U 1 1 5D1F2C92
 P 9000 5525
-F 0 "R701" H 9070 5571 50  0000 L CNN
+F 0 "R402" H 9070 5571 50  0000 L CNN
 F 1 "1K" H 9070 5480 50  0000 L CNN
 F 2 "Resistor_SMD:R_0402_1005Metric" V 8930 5525 50  0001 C CNN
@@
 	9000 5675 9000 5900
 $Comp
-L power:GND #PWR0108
+L power:GND #PWR0402
 U 1 1 5D1F308C
 P 9000 5900
-F 0 "#PWR0108" H 9000 5650 50  0001 C CNN
+F 0 "#PWR0402" H 9000 5650 50  0001 C CNN
 F 1 "GND" H 9005 5727 50  0000 C CNN
 F 2 "" H 9000 5900 50  0001 C CNN
@@
 $EndComp
 $Comp
-L Device:LED D704
+L Device:LED D403
 U 1 1 5D1F53AA
 P 9850 5050
-F 0 "D704" V 9889 4933 50  0000 R CNN
+F 0 "D403" V 9889 4933 50  0000 R CNN
 F 1 "LED" V 9798 4933 50  0000 R CNN
 F 2 "LED_SMD:LED_0402_1005Metric" H 9850 5050 50  0001 C CNN
@@
 $EndComp
 $Comp
-L Device:R R704
+L Device:R R403
 U 1 1 5D1F53B4
 P 9850 5525
-F 0 "R704" H 9920 5571 50  0000 L CNN
+F 0 "R403" H 9920 5571 50  0000 L CNN
 F 1 "1K" H 9920 5480 50  0000 L CNN
 F 2 "Resistor_SMD:R_0402_1005Metric" V 9780 5525 50  0001 C CNN
@@
 	9850 5675 9850 5900
 $Comp
-L power:GND #PWR0111
+L power:GND #PWR0403
 U 1 1 5D1F53C1
 P 9850 5900
-F 0 "#PWR0111" H 9850 5650 50  0001 C CNN
+F 0 "#PWR0403" H 9850 5650 50  0001 C CNN
 F 1 "GND" H 9855 5727 50  0000 C CNN
 F 2 "" H 9850 5900 50  0001 C CNN
@@
 $EndComp
 $Comp
-L Device:LED D705
+L Device:LED D404
 U 1 1 5D1F7859
 P 10275 5050
-F 0 "D705" V 10314 4933 50  0000 R CNN
+F 0 "D404" V 10314 4933 50  0000 R CNN
 F 1 "LED" V 10223 4933 50  0000 R CNN
 F 2 "LED_SMD:LED_0402_1005Metric" H 10275 5050 50  0001 C CNN
@@
 $EndComp
 $Comp
-L Device:R R705
+L Device:R R404
 U 1 1 5D1F7863
 P 10275 5525
-F 0 "R705" H 10345 5571 50  0000 L CNN
+F 0 "R404" H 10345 5571 50  0000 L CNN
 F 1 "1K" H 10345 5480 50  0000 L CNN
 F 2 "Resistor_SMD:R_0402_1005Metric" V 10205 5525 50  0001 C CNN
@@
 	10275 5675 10275 5900
 $Comp
-L power:GND #PWR0112
+L power:GND #PWR0404
 U 1 1 5D1F7870
 P 10275 5900
-F 0 "#PWR0112" H 10275 5650 50  0001 C CNN
+F 0 "#PWR0404" H 10275 5650 50  0001 C CNN
 F 1 "GND" H 10280 5727 50  0000 C CNN
 F 2 "" H 10275 5900 50  0001 C CNN
@@
 $EndComp
 $Comp
-L Device:LED D706
+L Device:LED D405
 U 1 1 5D1F787A
 P 10725 5050
-F 0 "D706" V 10764 4933 50  0000 R CNN
+F 0 "D405" V 10764 4933 50  0000 R CNN
 F 1 "LED" V 10673 4933 50  0000 R CNN
 F 2 "LED_SMD:LED_0402_1005Metric" H 10725 5050 50  0001 C CNN
@@
 $EndComp
 $Comp
-L Device:R R706
+L Device:R R405
 U 1 1 5D1F7884
 P 10725 5525
-F 0 "R706" H 10795 5571 50  0000 L CNN
+F 0 "R405" H 10795 5571 50  0000 L CNN
 F 1 "1K" H 10795 5480 50  0000 L CNN
 F 2 "Resistor_SMD:R_0402_1005Metric" V 10655 5525 50  0001 C CNN
@@
 	10725 5675 10725 5900
 $Comp
-L power:GND #PWR0113
+L power:GND #PWR0405
 U 1 1 5D1F7891
 P 10725 5900
-F 0 "#PWR0113" H 10725 5650 50  0001 C CNN
+F 0 "#PWR0405" H 10725 5650 50  0001 C CNN
 F 1 "GND" H 10730 5727 50  0000 C CNN
 F 2 "" H 10725 5900 50  0001 C CNN
@@
 	8550 4625 8550 4900
 $Comp
-L power:GND #PWR0109
+L power:GND #PWR0401
 U 1 1 5D1F3B22
 P 8550 5900
-F 0 "#PWR0109" H 8550 5650 50  0001 C CNN
+F 0 "#PWR0401" H 8550 5650 50  0001 C CNN
 F 1 "GND" H 8555 5727 50  0000 C CNN
 F 2 "" H 8550 5900 50  0001 C CNN
@@
 	8550 5200 8550 5375
 $Comp
-L Device:R R702
+L Device:R R401
 U 1 1 5D1F3B15
 P 8550 5525
-F 0 "R702" H 8620 5571 50  0000 L CNN
+F 0 "R401" H 8620 5571 50  0000 L CNN
 F 1 "1K" H 8620 5480 50  0000 L CNN
 F 2 "Resistor_SMD:R_0402_1005Metric" V 8480 5525 50  0001 C CNN
@@
 $EndComp
 $Comp
-L Device:LED D702
+L Device:LED D401
 U 1 1 5D1F3B0B
 P 8550 5050
-F 0 "D702" V 8589 4933 50  0000 R CNN
+F 0 "D401" V 8589 4933 50  0000 R CNN
 F 1 "LED" V 8498 4933 50  0000 R CNN
 F 2 "LED_SMD:LED_0402_1005Metric" H 8550 5050 50  0001 C CNN
