File: hw/LeashPCB/UserInputOutput.sch (KiCad schematic (older format))
At the start: 2 parts, among them SW1 SW_SPST, SW2 SW_SPST

Commit message: Adding part info for ordering components
Parts:
- SW1, SW2: Description (none) -> SWITCH TACTILE SPST-NO 0.05A 12V; Standard Price (none) -> $0.13050; Vendor1 (none) -> Panasonic Electronic Components
Changed lines of the file:
@@
 F 4 "EVQ-P7A01P" H 7900 4825 50  0001 C CNN "MPN1"
 F 5 "https://www.digikey.com/product-detail/en/panasonic-electronic-components/EVQ-P7A01P/P16763TR-ND/4429447" H 7900 4825 50  0001 C CNN "Link1"
+F 6 "SWITCH TACTILE SPST-NO 0.05A 12V" H 7900 4825 50  0001 C CNN "Description"
+F 7 "$0.13050	" H 7900 4825 50  0001 C CNN "Standard Price"
+F 8 "Panasonic Electronic Components" H 7900 4825 50  0001 C CNN "Vendor1"
 	1    7900 4825
 	1    0    0    -1
@@
 F 4 "EVQ-P7A01P" H 10125 4800 50  0001 C CNN "MPN1"
 F 5 "https://www.digikey.com/product-detail/en/panasonic-electronic-components/EVQ-P7A01P/P16763TR-ND/4429447" H 10125 4800 50  0001 C CNN "Link1"
+F 6 "SWITCH TACTILE SPST-NO 0.05A 12V" H 10125 4800 50  0001 C CNN "Description"
+F 7 "$0.13050	" H 10125 4800 50  0001 C CNN "Standard Price"
+F 8 "Panasonic Electronic Components" H 10125 4800 50  0001 C CNN "Vendor1"
 	1    10125 4800
 	1    0    0    -1

Commit message: Finished added components and generated BOM for ordering all parts
Parts:
- SW1, SW2: Short Description (none) -> SWITCH TACTILE SPST-NO 0.05A 12V
Changed lines of the file:
@@
 Sheet 6 10
 Title "BeagleDust Leash PCB"
-Date "2019-07-22"
-Rev "1"
+Date "2019-08-12"
+Rev "A"
 Comp "Beagleboard.org"
 Comment1 "Schematic designed by Analog Life, LLC"
@@
 F 7 "$0.13050	" H 7900 4825 50  0001 C CNN "Standard Price"
 F 8 "Panasonic Electronic Components" H 7900 4825 50  0001 C CNN "Vendor1"
+F 9 "SWITCH TACTILE SPST-NO 0.05A 12V" H 7900 4825 50  0001 C CNN "Short Description"
 	1    7900 4825
 	1    0    0    -1
@@
 F 7 "$0.13050	" H 10125 4800 50  0001 C CNN "Standard Price"
 F 8 "Panasonic Electronic Components" H 10125 4800 50  0001 C CNN "Vendor1"
+F 9 "SWITCH TACTILE SPST-NO 0.05A 12V" H 10125 4800 50  0001 C CNN "Short Description"
 	1    10125 4800
 	1    0    0    -1

Commit message: Swapped out USB and antenna sections and refactored outline, started routing
Parts:
- SW1, SW2: footprint leash:EVQ-P7A01P -> Button_Switch_SMD:SW_SPST_PTS810
Changed lines of the file:
@@
 EESchema Schematic File Version 4
-LIBS:LeashPCB-cache
 EELAYER 30 0
 EELAYER END
 $Descr B 17000 11000
 encoding utf-8
-Sheet 6 10
+Sheet 5 9
 Title "BeagleDust Leash PCB"
 Date "2019-08-12"
@@
 F 0 "SW2" H 7900 5060 50  0000 C CNN
 F 1 "SW_SPST" H 7900 4969 50  0000 C CNN
-F 2 "leash:EVQ-P7A01P" H 7900 4825 50  0001 C CNN
+F 2 "Button_Switch_SMD:SW_SPST_PTS810" H 7900 4825 50  0001 C CNN
 F 3 "https://b2b-api.panasonic.eu/file_stream/pids/fileversion/2431" H 7900 4825 50  0001 C CNN
 F 4 "EVQ-P7A01P" H 7900 4825 50  0001 C CNN "MPN1"
@@
 F 0 "SW1" H 10125 5035 50  0000 C CNN
 F 1 "SW_SPST" H 10125 4944 50  0000 C CNN
-F 2 "leash:EVQ-P7A01P" H 10125 4800 50  0001 C CNN
+F 2 "Button_Switch_SMD:SW_SPST_PTS810" H 10125 4800 50  0001 C CNN
 F 3 "https://b2b-api.panasonic.eu/file_stream/pids/fileversion/2431" H 10125 4800 50  0001 C CNN
 F 4 "EVQ-P7A01P" H 10125 4800 50  0001 C CNN "MPN1"

Commit message: Done with 90% of routing, but going to move the USB to serial and power chips to open up the pathways underneath the CC1352R
Parts:
- removed SW1, SW2: SW_SPST, Button_Switch_SMD:SW_SPST_PTS810, symbol Switch:SW_SPST
- added SW901, SW902: SW_SPST, Button_Switch_SMD:SW_SPST_PTS810, symbol Switch:SW_SPST
Connections:
- net labels added: RESET_N, USER
- net labels removed: RST_BTN, USER_BTN
Changed lines of the file:
@@
 $Descr B 17000 11000
 encoding utf-8
-Sheet 5 9
+Sheet 9 9
 Title "BeagleDust Leash PCB"
 Date "2019-08-12"
@@
 $EndDescr
 $Comp
-L Switch:SW_SPST SW2
-U 1 1 5D565CF9
-P 7900 4825
-F 0 "SW2" H 7900 5060 50  0000 C CNN
-F 1 "SW_SPST" H 7900 4969 50  0000 C CNN
-F 2 "Button_Switch_SMD:SW_SPST_PTS810" H 7900 4825 50  0001 C CNN
-F 3 "https://b2b-api.panasonic.eu/file_stream/pids/fileversion/2431" H 7900 4825 50  0001 C CNN
-F 4 "EVQ-P7A01P" H 7900 4825 50  0001 C CNN "MPN1"
-F 5 "https://www.digikey.com/product-detail/en/panasonic-electronic-components/EVQ-P7A01P/P16763TR-ND/4429447" H 7900 4825 50  0001 C CNN "Link1"
-F 6 "SWITCH TACTILE SPST-NO 0.05A 12V" H 7900 4825 50  0001 C CNN "Description"
-F 7 "$0.13050	" H 7900 4825 50  0001 C CNN "Standard Price"
-F 8 "Panasonic Electronic Components" H 7900 4825 50  0001 C CNN "Vendor1"
-F 9 "SWITCH TACTILE SPST-NO 0.05A 12V" H 7900 4825 50  0001 C CNN "Short Description"
-	1    7900 4825
+L Switch:SW_SPST SW901
+U 1 1 5E6BAEE4
+P 7250 5425
+F 0 "SW901" H 7250 5660 50  0000 C CNN
+F 1 "SW_SPST" H 7250 5569 50  0000 C CNN
+F 2 "Button_Switch_SMD:SW_SPST_PTS810" H 7250 5425 50  0001 C CNN
+F 3 "https://b2b-api.panasonic.eu/file_stream/pids/fileversion/2431" H 7250 5425 50  0001 C CNN
+F 4 "EVQ-P7A01P" H 7250 5425 50  0001 C CNN "MPN1"
+F 5 "https://www.digikey.com/product-detail/en/panasonic-electronic-components/EVQ-P7A01P/P16763TR-ND/4429447" H 7250 5425 50  0001 C CNN "Link1"
+F 6 "SWITCH TACTILE SPST-NO 0.05A 12V" H 7250 5425 50  0001 C CNN "Description"
+F 7 "$0.13050	" H 7250 5425 50  0001 C CNN "Standard Price"
+F 8 "Panasonic Electronic Components" H 7250 5425 50  0001 C CNN "Vendor1"
+F 9 "SWITCH TACTILE SPST-NO 0.05A 12V" H 7250 5425 50  0001 C CNN "Short Description"
+	1    7250 5425
 	1    0    0    -1
 $EndComp
 $Comp
-L power:GND #PWR0103
-U 1 1 5D565FA6
-P 8200 5200
-F 0 "#PWR0103" H 8200 4950 50  0001 C CNN
-F 1 "GND" H 8205 5027 50  0000 C CNN
-F 2 "" H 8200 5200 50  0001 C CNN
-F 3 "" H 8200 5200 50  0001 C CNN
-	1    8200 5200
+L power:GND #PWR0901
+U 1 1 5E6BAEEA
+P 7550 5800
+F 0 "#PWR0901" H 7550 5550 50  0001 C CNN
+F 1 "GND" H 7555 5627 50  0000 C CNN
+F 2 "" H 7550 5800 50  0001 C CNN
+F 3 "" H 7550 5800 50  0001 C CNN
+	1    7550 5800
 	1    0    0    -1
 $EndComp
 Wire Wire Line
-	8200 5200 8200 4825
+	7550 5800 7550 5425
 Wire Wire Line
-	8200 4825 8100 4825
+	7550 5425 7450 5425
 $Comp
-L Switch:SW_SPST SW1
-U 1 1 5D568EA2
-P 10125 4800
-F 0 "SW1" H 10125 5035 50  0000 C CNN
-F 1 "SW_SPST" H 10125 4944 50  0000 C CNN
-F 2 "Button_Switch_SMD:SW_SPST_PTS810" H 10125 4800 50  0001 C CNN
-F 3 "https://b2b-api.panasonic.eu/file_stream/pids/fileversion/2431" H 10125 4800 50  0001 C CNN
-F 4 "EVQ-P7A01P" H 10125 4800 50  0001 C CNN "MPN1"
-F 5 "https://www.digikey.com/product-detail/en/panasonic-electronic-components/EVQ-P7A01P/P16763TR-ND/4429447" H 10125 4800 50  0001 C CNN "Link1"
-F 6 "SWITCH TACTILE SPST-NO 0.05A 12V" H 10125 4800 50  0001 C CNN "Description"
-F 7 "$0.13050	" H 10125 4800 50  0001 C CNN "Standard Price"
-F 8 "Panasonic Electronic Components" H 10125 4800 50  0001 C CNN "Vendor1"
-F 9 "SWITCH TACTILE SPST-NO 0.05A 12V" H 10125 4800 50  0001 C CNN "Short Description"
-	1    10125 4800
+L Switch:SW_SPST SW902
+U 1 1 5E6BAEF8
+P 9475 5400
+F 0 "SW902" H 9475 5635 50  0000 C CNN
+F 1 "SW_SPST" H 9475 5544 50  0000 C CNN
+F 2 "Button_Switch_SMD:SW_SPST_PTS810" H 9475 5400 50  0001 C CNN
+F 3 "https://b2b-api.panasonic.eu/file_stream/pids/fileversion/2431" H 9475 5400 50  0001 C CNN
+F 4 "EVQ-P7A01P" H 9475 5400 50  0001 C CNN "MPN1"
+F 5 "https://www.digikey.com/product-detail/en/panasonic-electronic-components/EVQ-P7A01P/P16763TR-ND/4429447" H 9475 5400 50  0001 C CNN "Link1"
+F 6 "SWITCH TACTILE SPST-NO 0.05A 12V" H 9475 5400 50  0001 C CNN "Description"
+F 7 "$0.13050	" H 9475 5400 50  0001 C CNN "Standard Price"
+F 8 "Panasonic Electronic Components" H 9475 5400 50  0001 C CNN "Vendor1"
+F 9 "SWITCH TACTILE SPST-NO 0.05A 12V" H 9475 5400 50  0001 C CNN "Short Description"
+	1    9475 5400
 	1    0    0    -1
 $EndComp
 $Comp
-L power:GND #PWR0153
-U 1 1 5D568EAC
-P 10425 5175
-F 0 "#PWR0153" H 10425 4925 50  0001 C CNN
-F 1 "GND" H 10430 5002 50  0000 C CNN
-F 2 "" H 10425 5175 50  0001 C CNN
-F 3 "" H 10425 5175 50  0001 C CNN
-	1    10425 5175
+L power:GND #PWR0902
+U 1 1 5E6BAEFE
+P 9775 5775
+F 0 "#PWR0902" H 9775 5525 50  0001 C CNN
+F 1 "GND" H 9780 5602 50  0000 C CNN
+F 2 "" H 9775 5775 50  0001 C CNN
+F 3 "" H 9775 5775 50  0001 C CNN
+	1    9775 5775
 	1    0    0    -1
 $EndComp
 Wire Wire Line
-	10425 5175 10425 4800
+	9775 5775 9775 5400
 Wire Wire Line
-	10425 4800 10325 4800
+	9775 5400 9675 5400
 Wire Wire Line
-	9925 4800 9675 4800
-Text HLabel 7325 4825 0    98   Input ~ 0
-RST_BTN
+	9275 5400 9025 5400
 Wire Wire Line
-	7325 4825 7700 4825
-Text HLabel 9675 4800 0    98   Input ~ 0
-USER_BTN
+	6675 5425 7050 5425
+Text GLabel 6675 5425 0    79   Input ~ 0
+RESET_N
+Text GLabel 9025 5400 0    79   Input ~ 0
+USER
 $EndSCHEMATC

Commit message: Migrated all hierarchical labels to global labels
Parts:
- added C906, C907: 0.1 uF, Capacitor_SMD:C_0402_1005Metric, symbol Device:C
- added R901, R902: 100K, Resistor_SMD:R_0402_1005Metric, symbol Device:R
Connections:
- net labels added: USER1, VDDS
- net labels removed: USER
- wire segments 6 -> 20
Changed lines of the file:
@@
 L Switch:SW_SPST SW901
 U 1 1 5E6BAEE4
-P 7250 5425
-F 0 "SW901" H 7250 5660 50  0000 C CNN
-F 1 "SW_SPST" H 7250 5569 50  0000 C CNN
-F 2 "Button_Switch_SMD:SW_SPST_PTS810" H 7250 5425 50  0001 C CNN
-F 3 "https://b2b-api.panasonic.eu/file_stream/pids/fileversion/2431" H 7250 5425 50  0001 C CNN
-F 4 "EVQ-P7A01P" H 7250 5425 50  0001 C CNN "MPN1"
-F 5 "https://www.digikey.com/product-detail/en/panasonic-electronic-components/EVQ-P7A01P/P16763TR-ND/4429447" H 7250 5425 50  0001 C CNN "Link1"
-F 6 "SWITCH TACTILE SPST-NO 0.05A 12V" H 7250 5425 50  0001 C CNN "Description"
-F 7 "$0.13050	" H 7250 5425 50  0001 C CNN "Standard Price"
-F 8 "Panasonic Electronic Components" H 7250 5425 50  0001 C CNN "Vendor1"
-F 9 "SWITCH TACTILE SPST-NO 0.05A 12V" H 7250 5425 50  0001 C CNN "Short Description"
-	1    7250 5425
+P 6575 5450
+F 0 "SW901" H 6575 5685 50  0000 C CNN
+F 1 "SW_SPST" H 6575 5594 50  0000 C CNN
+F 2 "Button_Switch_SMD:SW_SPST_PTS810" H 6575 5450 50  0001 C CNN
+F 3 "https://b2b-api.panasonic.eu/file_stream/pids/fileversion/2431" H 6575 5450 50  0001 C CNN
+F 4 "EVQ-P7A01P" H 6575 5450 50  0001 C CNN "MPN1"
+F 5 "https://www.digikey.com/product-detail/en/panasonic-electronic-components/EVQ-P7A01P/P16763TR-ND/4429447" H 6575 5450 50  0001 C CNN "Link1"
+F 6 "SWITCH TACTILE SPST-NO 0.05A 12V" H 6575 5450 50  0001 C CNN "Description"
+F 7 "$0.13050	" H 6575 5450 50  0001 C CNN "Standard Price"
+F 8 "Panasonic Electronic Components" H 6575 5450 50  0001 C CNN "Vendor1"
+F 9 "SWITCH TACTILE SPST-NO 0.05A 12V" H 6575 5450 50  0001 C CNN "Short Description"
+	1    6575 5450
 	1    0    0    -1
 $EndComp
@@
 L power:GND #PWR0901
 U 1 1 5E6BAEEA
-P 7550 5800
-F 0 "#PWR0901" H 7550 5550 50  0001 C CNN
-F 1 "GND" H 7555 5627 50  0000 C CNN
-F 2 "" H 7550 5800 50  0001 C CNN
-F 3 "" H 7550 5800 50  0001 C CNN
-	1    7550 5800
-	1    0    0    -1
-$EndComp
-Wire Wire Line
-	7550 5800 7550 5425
-Wire Wire Line
-	7550 5425 7450 5425
+P 6875 5825
+F 0 "#PWR0901" H 6875 5575 50  0001 C CNN
+F 1 "GND" H 6880 5652 50  0000 C CNN
+F 2 "" H 6875 5825 50  0001 C CNN
+F 3 "" H 6875 5825 50  0001 C CNN
+	1    6875 5825
+	1    0    0    -1
+$EndComp
+Wire Wire Line
+	6875 5825 6875 5450
+Wire Wire Line
+	6875 5450 6775 5450
 $Comp
 L Switch:SW_SPST SW902
 U 1 1 5E6BAEF8
-P 9475 5400
-F 0 "SW902" H 9475 5635 50  0000 C CNN
-F 1 "SW_SPST" H 9475 5544 50  0000 C CNN
-F 2 "Button_Switch_SMD:SW_SPST_PTS810" H 9475 5400 50  0001 C CNN
-F 3 "https://b2b-api.panasonic.eu/file_stream/pids/fileversion/2431" H 9475 5400 50  0001 C CNN
-F 4 "EVQ-P7A01P" H 9475 5400 50  0001 C CNN "MPN1"
-F 5 "https://www.digikey.com/product-detail/en/panasonic-electronic-components/EVQ-P7A01P/P16763TR-ND/4429447" H 9475 5400 50  0001 C CNN "Link1"
-F 6 "SWITCH TACTILE SPST-NO 0.05A 12V" H 9475 5400 50  0001 C CNN "Description"
-F 7 "$0.13050	" H 9475 5400 50  0001 C CNN "Standard Price"
-F 8 "Panasonic Electronic Components" H 9475 5400 50  0001 C CNN "Vendor1"
-F 9 "SWITCH TACTILE SPST-NO 0.05A 12V" H 9475 5400 50  0001 C CNN "Short Description"
-	1    9475 5400
+P 9075 5400
+F 0 "SW902" H 9075 5635 50  0000 C CNN
+F 1 "SW_SPST" H 9075 5544 50  0000 C CNN
+F 2 "Button_Switch_SMD:SW_SPST_PTS810" H 9075 5400 50  0001 C CNN
+F 3 "https://b2b-api.panasonic.eu/file_stream/pids/fileversion/2431" H 9075 5400 50  0001 C CNN
+F 4 "EVQ-P7A01P" H 9075 5400 50  0001 C CNN "MPN1"
+F 5 "https://www.digikey.com/product-detail/en/panasonic-electronic-components/EVQ-P7A01P/P16763TR-ND/4429447" H 9075 5400 50  0001 C CNN "Link1"
+F 6 "SWITCH TACTILE SPST-NO 0.05A 12V" H 9075 5400 50  0001 C CNN "Description"
+F 7 "$0.13050	" H 9075 5400 50  0001 C CNN "Standard Price"
+F 8 "Panasonic Electronic Components" H 9075 5400 50  0001 C CNN "Vendor1"
+F 9 "SWITCH TACTILE SPST-NO 0.05A 12V" H 9075 5400 50  0001 C CNN "Short Description"
+	1    9075 5400
 	1    0    0    -1
 $EndComp
@@
 L power:GND #PWR0902
 U 1 1 5E6BAEFE
-P 9775 5775
-F 0 "#PWR0902" H 9775 5525 50  0001 C CNN
-F 1 "GND" H 9780 5602 50  0000 C CNN
-F 2 "" H 9775 5775 50  0001 C CNN
-F 3 "" H 9775 5775 50  0001 C CNN
-	1    9775 5775
-	1    0    0    -1
-$EndComp
-Wire Wire Line
-	9775 5775 9775 5400
-Wire Wire Line
-	9775 5400 9675 5400
-Wire Wire Line
-	9275 5400 9025 5400
-Wire Wire Line
-	6675 5425 7050 5425
-Text GLabel 6675 5425 0    79   Input ~ 0
+P 9375 5775
+F 0 "#PWR0902" H 9375 5525 50  0001 C CNN
+F 1 "GND" H 9380 5602 50  0000 C CNN
+F 2 "" H 9375 5775 50  0001 C CNN
+F 3 "" H 9375 5775 50  0001 C CNN
+	1    9375 5775
+	1    0    0    -1
+$EndComp
+Wire Wire Line
+	9375 5775 9375 5400
+Wire Wire Line
+	9375 5400 9275 5400
+Text GLabel 5675 5550 0    79   Input ~ 0
 RESET_N
-Text GLabel 9025 5400 0    79   Input ~ 0
-USER
+Wire Wire Line
+	5900 5550 5900 5575
+Wire Wire Line
+	5675 5550 5900 5550
+Connection ~ 5900 5550
+Wire Wire Line
+	5900 5450 5900 5550
+$Comp
+L power:GND #PWR?
+U 1 1 5E811A57
+P 5900 6050
+AR Path="/5D062750/5E811A57" Ref="#PWR?"  Part="1"
+AR Path="/5D099F4C/5E811A57" Ref="#PWR0123"  Part="1"
+F 0 "#PWR0123" H 5900 5800 50  0001 C CNN
+F 1 "GND" H 5905 5877 50  0000 C CNN
+F 2 "" H 5900 6050 50  0001 C CNN
+F 3 "" H 5900 6050 50  0001 C CNN
+	1    5900 6050
+	1    0    0    -1
+$EndComp
+Connection ~ 5900 5450
+Wire Wire Line
+	5900 5400 5900 5450
+Wire Wire Line
+	5900 5875 5900 6050
+Wire Wire Line
+	5900 5000 5900 5100
+Wire Wire Line
+	5650 5000 5900 5000
+$Comp
+L Device:R R?
+U 1 1 5E811A69
+P 5900 5250
+AR Path="/5D062750/5E811A69" Ref="R?"  Part="1"
+AR Path="/5D099F4C/5E811A69" Ref="R901"  Part="1"
+F 0 "R901" H 5970 5296 50  0000 L CNN
+F 1 "100K" H 5970 5205 50  0000 L CNN
+F 2 "Resistor_SMD:R_0402_1005Metric" V 5830 5250 50  0001 C CNN
+F 3 "~" H 5900 5250 50  0001 C CNN
+F 4 "RES SMD 100K OHM 5% 1/16W 0402" H 5900 5250 50  0001 C CNN "Description"
+F 5 "https://www.digikey.com/product-detail/en/yageo/RC0402JR-07100KL/311-100KJRCT-ND/729363" H 5900 5250 50  0001 C CNN "Link1"
+F 6 "RC0402JR-07100KL" H 5900 5250 50  0001 C CNN "MPN1"
+F 7 "$0.00139" H 5900 5250 50  0001 C CNN "Standard Price"
+F 8 "Yageo" H 5900 5250 50  0001 C CNN "Vendor1"
+F 9 "RES SMD 100K OHM 5% 1/16W 0402" H 5900 5250 50  0001 C CNN "Short Description"
+	1    5900 5250
+	1    0    0    -1
+$EndComp
+$Comp
+L Device:C C?
+U 1 1 5E811A75
+P 5900 5725
+AR Path="/5D062750/5E811A75" Ref="C?"  Part="1"
+AR Path="/5D099F4C/5E811A75" Ref="C906"  Part="1"
+F 0 "C906" H 5785 5679 50  0000 R CNN
+F 1 "0.1 uF" H 5785 5770 50  0000 R CNN
+F 2 "Capacitor_SMD:C_0402_1005Metric" H 5938 5575 50  0001 C CNN
+F 3 "~" H 5900 5725 50  0001 C CNN
+F 4 "CAP CER 0.1UF 10V X5R 0402" H 5900 5725 50  0001 C CNN "Description"
+F 5 "https://www.digikey.com/product-detail/en/samsung-electro-mechanics/CL05A104MP5NNNC/1276-1443-1-ND/3889529" H 5900 5725 50  0001 C CNN "Link1"
+F 6 "CL05A104MP5NNNC" H 5900 5725 50  0001 C CNN "MPN1"
+F 7 "$0.00315" H 5900 5725 50  0001 C CNN "Standard Price"
+F 8 "Samsung Electro-Mechanics" H 5900 5725 50  0001 C CNN "Vendor1"
+F 9 "CAP CER 0.1UF 10V X5R 0402" H 5900 5725 50  0001 C CNN "Short Description"
+	1    5900 5725
+	-1   0    0    1
+$EndComp
+Wire Wire Line
+	5900 5450 6375 5450
+Text GLabel 5650 5000 0    63   Input ~ 0
+VDDS
+Text GLabel 8300 5500 0    79   Input ~ 0
+USER1
+Wire Wire Line
+	8525 5500 8525 5525
+Wire Wire Line
+	8300 5500 8525 5500
+Connection ~ 8525 5500
+Wire Wire Line
+	8525 5400 8525 5500
+$Comp
+L power:GND #PWR?
+U 1 1 5E815CF5
+P 8525 6000
+AR Path="/5D062750/5E815CF5" Ref="#PWR?"  Part="1"
+AR Path="/5D099F4C/5E815CF5" Ref="#PWR0124"  Part="1"
+F 0 "#PWR0124" H 8525 5750 50  0001 C CNN
+F 1 "GND" H 8530 5827 50  0000 C CNN
+F 2 "" H 8525 6000 50  0001 C CNN
+F 3 "" H 8525 6000 50  0001 C CNN
+	1    8525 6000
+	1    0    0    -1
+$EndComp
+Connection ~ 8525 5400
+Wire Wire Line
+	8525 5350 8525 5400
+Wire Wire Line
+	8525 5825 8525 6000
+Wire Wire Line
+	8525 4950 8525 5050
+Wire Wire Line
+	8275 4950 8525 4950
+$Comp
+L Device:R R?
+U 1 1 5E815D0A
+P 8525 5200
+AR Path="/5D062750/5E815D0A" Ref="R?"  Part="1"
+AR Path="/5D099F4C/5E815D0A" Ref="R902"  Part="1"
+F 0 "R902" H 8595 5246 50  0000 L CNN
+F 1 "100K" H 8595 5155 50  0000 L CNN
+F 2 "Resistor_SMD:R_0402_1005Metric" V 8455 5200 50  0001 C CNN
+F 3 "~" H 8525 5200 50  0001 C CNN
+F 4 "RES SMD 100K OHM 5% 1/16W 0402" H 8525 5200 50  0001 C CNN "Description"
+F 5 "https://www.digikey.com/product-detail/en/yageo/RC0402JR-07100KL/311-100KJRCT-ND/729363" H 8525 5200 50  0001 C CNN "Link1"
+F 6 "RC0402JR-07100KL" H 8525 5200 50  0001 C CNN "MPN1"
+F 7 "$0.00139" H 8525 5200 50  0001 C CNN "Standard Price"
+F 8 "Yageo" H 8525 5200 50  0001 C CNN "Vendor1"
+F 9 "RES SMD 100K OHM 5% 1/16W 0402" H 8525 5200 50  0001 C CNN "Short Description"
+	1    8525 5200
+	1    0    0    -1
+$EndComp
+$Comp
+L Device:C C?
+U 1 1 5E815D1A
+P 8525 5675
+AR Path="/5D062750/5E815D1A" Ref="C?"  Part="1"
+AR Path="/5D099F4C/5E815D1A" Ref="C907"  Part="1"
+F 0 "C907" H 8410 5629 50  0000 R CNN
+F 1 "0.1 uF" H 8410 5720 50  0000 R CNN
+F 2 "Capacitor_SMD:C_0402_1005Metric" H 8563 5525 50  0001 C CNN
+F 3 "~" H 8525 5675 50  0001 C CNN
+F 4 "CAP CER 0.1UF 10V X5R 0402" H 8525 5675 50  0001 C CNN "Description"
+F 5 "https://www.digikey.com/product-detail/en/samsung-electro-mechanics/CL05A104MP5NNNC/1276-1443-1-ND/3889529" H 8525 5675 50  0001 C CNN "Link1"
+F 6 "CL05A104MP5NNNC" H 8525 5675 50  0001 C CNN "MPN1"
+F 7 "$0.00315" H 8525 5675 50  0001 C CNN "Standard Price"
+F 8 "Samsung Electro-Mechanics" H 8525 5675 50  0001 C CNN "Vendor1"
+F 9 "CAP CER 0.1UF 10V X5R 0402" H 8525 5675 50  0001 C CNN "Short Description"
+	1    8525 5675
+	-1   0    0    1
+$EndComp
+Text GLabel 8275 4950 0    63   Input ~ 0
+VDDS
+Wire Wire Line
+	8525 5400 8875 5400
 $EndSCHEMATC

Commit message: Removed two extra pullup resistors
Parts:
- renumbered C906 to C901, C907 to C902
Changed lines of the file:
@@
 $EndComp
 $Comp
-L power:GND #PWR0901
+L power:GND #PWR0902
 U 1 1 5E6BAEEA
 P 6875 5825
-F 0 "#PWR0901" H 6875 5575 50  0001 C CNN
+F 0 "#PWR0902" H 6875 5575 50  0001 C CNN
 F 1 "GND" H 6880 5652 50  0000 C CNN
 F 2 "" H 6875 5825 50  0001 C CNN
@@
 $EndComp
 $Comp
-L power:GND #PWR0902
+L power:GND #PWR0904
 U 1 1 5E6BAEFE
 P 9375 5775
-F 0 "#PWR0902" H 9375 5525 50  0001 C CNN
+F 0 "#PWR0904" H 9375 5525 50  0001 C CNN
 F 1 "GND" H 9380 5602 50  0000 C CNN
 F 2 "" H 9375 5775 50  0001 C CNN
@@
 P 5900 6050
 AR Path="/5D062750/5E811A57" Ref="#PWR?"  Part="1"
-AR Path="/5D099F4C/5E811A57" Ref="#PWR0123"  Part="1"
-F 0 "#PWR0123" H 5900 5800 50  0001 C CNN
+AR Path="/5D099F4C/5E811A57" Ref="#PWR0901"  Part="1"
+F 0 "#PWR0901" H 5900 5800 50  0001 C CNN
 F 1 "GND" H 5905 5877 50  0000 C CNN
 F 2 "" H 5900 6050 50  0001 C CNN
@@
 P 5900 5725
 AR Path="/5D062750/5E811A75" Ref="C?"  Part="1"
-AR Path="/5D099F4C/5E811A75" Ref="C906"  Part="1"
-F 0 "C906" H 5785 5679 50  0000 R CNN
+AR Path="/5D099F4C/5E811A75" Ref="C901"  Part="1"
+F 0 "C901" H 5785 5679 50  0000 R CNN
 F 1 "0.1 uF" H 5785 5770 50  0000 R CNN
 F 2 "Capacitor_SMD:C_0402_1005Metric" H 5938 5575 50  0001 C CNN
@@
 P 8525 6000
 AR Path="/5D062750/5E815CF5" Ref="#PWR?"  Part="1"
-AR Path="/5D099F4C/5E815CF5" Ref="#PWR0124"  Part="1"
-F 0 "#PWR0124" H 8525 5750 50  0001 C CNN
+AR Path="/5D099F4C/5E815CF5" Ref="#PWR0903"  Part="1"
+F 0 "#PWR0903" H 8525 5750 50  0001 C CNN
 F 1 "GND" H 8530 5827 50  0000 C CNN
 F 2 "" H 8525 6000 50  0001 C CNN
@@
 P 8525 5675
 AR Path="/5D062750/5E815D1A" Ref="C?"  Part="1"
-AR Path="/5D099F4C/5E815D1A" Ref="C907"  Part="1"
-F 0 "C907" H 8410 5629 50  0000 R CNN
+AR Path="/5D099F4C/5E815D1A" Ref="C902"  Part="1"
+F 0 "C902" H 8410 5629 50  0000 R CNN
 F 1 "0.1 uF" H 8410 5720 50  0000 R CNN
 F 2 "Capacitor_SMD:C_0402_1005Metric" H 8563 5525 50  0001 C CNN
