File: hw/LeashPCB/UserInputOutput.sch (KiCad schematic (older format))
At the start: 6 parts, among them SW901 SW_SPST, SW902 SW_SPST

Commit message: Updated BOM for ordering parts
Parts:
- SW901, SW902: Link1 https://www.digikey.com/product-detail/en/panasonic-electro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 -> https://www.seeedstudio.com/opl.html; Link2 (none) -> https://www.digikey.com/product-detail/en/panasonic-electro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; MPN1 EVQ-P7A01P -> SKRPABE010; MPN2 (none) -> EVQ-P7A01P; Vendor1 Panasonic Electronic Components -> ALPS; Vendor2 (none) -> Panasonic Electronic Components
Changed lines of the file:
@@
 F 2 "Button_Switch_SMD:SW_SPST_PTS810" H 6575 5450 50  0001 C CNN
 F 3 "https://b2b-api.panasonic.eu/file_stream/pids/fileversion/2431" H 6575 5450 50  0001 C CNN
-F 4 "EVQ-P7A01P" H 6575 5450 50  0001 C CNN "MPN1"
-F 5 "https://www.digikey.com/product-detail/en/panasonic-electronic-components/EVQ-P7A01P/P16763TR-ND/4429447" H 6575 5450 50  0001 C CNN "Link1"
+F 4 "SKRPABE010" H 6575 5450 50  0001 C CNN "MPN1"
+F 5 "https://www.seeedstudio.com/opl.html" H 6575 5450 50  0001 C CNN "Link1"
 F 6 "SWITCH TACTILE SPST-NO 0.05A 12V" H 6575 5450 50  0001 C CNN "Description"
 F 7 "$0.13050	" H 6575 5450 50  0001 C CNN "Standard Price"
-F 8 "Panasonic Electronic Components" H 6575 5450 50  0001 C CNN "Vendor1"
+F 8 "ALPS" H 6575 5450 50  0001 C CNN "Vendor1"
 F 9 "SWITCH TACTILE SPST-NO 0.05A 12V" H 6575 5450 50  0001 C CNN "Short Description"
+F 10 "https://www.digikey.com/product-detail/en/panasonic-electronic-components/EVQ-P7A01P/P16763TR-ND/4429447" H 6575 5450 50  0001 C CNN "Link2"
+F 11 "EVQ-P7A01P" H 6575 5450 50  0001 C CNN "MPN2"
+F 12 "Panasonic Electronic Components" H 6575 5450 50  0001 C CNN "Vendor2"
 	1    6575 5450
 	1    0    0    -1
@@
 F 2 "Button_Switch_SMD:SW_SPST_PTS810" H 9075 5400 50  0001 C CNN
 F 3 "https://b2b-api.panasonic.eu/file_stream/pids/fileversion/2431" H 9075 5400 50  0001 C CNN
-F 4 "EVQ-P7A01P" H 9075 5400 50  0001 C CNN "MPN1"
-F 5 "https://www.digikey.com/product-detail/en/panasonic-electronic-components/EVQ-P7A01P/P16763TR-ND/4429447" H 9075 5400 50  0001 C CNN "Link1"
+F 4 "SKRPABE010" H 9075 5400 50  0001 C CNN "MPN1"
+F 5 "https://www.seeedstudio.com/opl.html" H 9075 5400 50  0001 C CNN "Link1"
 F 6 "SWITCH TACTILE SPST-NO 0.05A 12V" H 9075 5400 50  0001 C CNN "Description"
 F 7 "$0.13050	" H 9075 5400 50  0001 C CNN "Standard Price"
-F 8 "Panasonic Electronic Components" H 9075 5400 50  0001 C CNN "Vendor1"
+F 8 "ALPS" H 9075 5400 50  0001 C CNN "Vendor1"
 F 9 "SWITCH TACTILE SPST-NO 0.05A 12V" H 9075 5400 50  0001 C CNN "Short Description"
+F 10 "https://www.digikey.com/product-detail/en/panasonic-electronic-components/EVQ-P7A01P/P16763TR-ND/4429447" H 9075 5400 50  0001 C CNN "Link2"
+F 11 "EVQ-P7A01P" H 9075 5400 50  0001 C CNN "MPN2"
+F 12 "Panasonic Electronic Components" H 9075 5400 50  0001 C CNN "Vendor2"
 	1    9075 5400
 	1    0    0    -1
