File: hw/LeashPCB/ExternalInput.sch (KiCad schematic (older format))
At the start: 2 parts, among them J301 Conn_01x02_Male

Commit message: Adding part info for ordering components
Parts:
- D301: Description (none) -> DIODE SCHOTTKY 30V 200MA SOD123; Link1 (none) -> https://www.digikey.com/product-detail/en/nexperia-usa-inc/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; MPN1 (none) -> BAT54GWJ; Standard Price (none) -> $0.02037; Vendor1 (none) -> Nexperia USA Inc.
- J301: Description (none) -> CONN HEADER SMD R/A 2POS 2MM; Link1 https://lcsc.com/product-detail/Wire-To-Board-Wire-To-Wire-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 -> https://www.digikey.com/product-detail/en/jst-sales-america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; MPN1 (none) -> S2B-PH-SM4-TB(LF)(SN); Standard Price 0.03 -> $0.03; Vendor1 (none) -> JST Sales America Inc.
Changed lines of the file:
@@
 F 2 "Connector_JST:JST_PH_S2B-PH-SM4-TB_1x02-1MP_P2.00mm_Horizontal" H 7500 4725 50  0001 C CNN
 F 3 "~" H 7500 4725 50  0001 C CNN
-F 4 "0.03" H 7500 4725 50  0001 C CNN "Standard Price"
-F 5 "https://lcsc.com/product-detail/Wire-To-Board-Wire-To-Wire-Connector_Boom-Precision-Elec-PH2-0-2PWB-2P-pitch2-0mm-Horizontal_C47647.html" H 7500 4725 50  0001 C CNN "Link1"
+F 4 "$0.03" H 7500 4725 50  0001 C CNN "Standard Price"
+F 5 "https://www.digikey.com/product-detail/en/jst-sales-america-inc/S2B-PH-SM4-TB-LF-SN/455-1749-1-ND/926846" H 7500 4725 50  0001 C CNN "Link1"
+F 6 "CONN HEADER SMD R/A 2POS 2MM" H 7500 4725 50  0001 C CNN "Description"
+F 7 "S2B-PH-SM4-TB(LF)(SN)" H 7500 4725 50  0001 C CNN "MPN1"
+F 8 "JST Sales America Inc." H 7500 4725 50  0001 C CNN "Vendor1"
 	1    7500 4725
 	1    0    0    -1
@@
 F 2 "Diode_SMD:D_SOD-123" H 8750 4550 50  0001 C CNN
 F 3 "" H 8750 4725 50  0001 C CNN
+F 4 "DIODE SCHOTTKY 30V 200MA SOD123" H 8750 4725 50  0001 C CNN "Description"
+F 5 "https://www.digikey.com/product-detail/en/nexperia-usa-inc/BAT54GWJ/1727-7328-1-ND/7390579" H 8750 4725 50  0001 C CNN "Link1"
+F 6 "BAT54GWJ" H 8750 4725 50  0001 C CNN "MPN1"
+F 7 "$0.02037" H 8750 4725 50  0001 C CNN "Standard Price"
+F 8 "Nexperia USA Inc." H 8750 4725 50  0001 C CNN "Vendor1"
 	1    8750 4725
 	-1   0    0    1

Commit message: Finished added components and generated BOM for ordering all parts
Parts:
- D301: Short Description (none) -> DIODE SCHOTTKY 30V 200MA SOD123
- J301: Short Description (none) -> CONN HEADER SMD R/A 2POS 2MM
Changed lines of the file:
@@
 Sheet 3 10
 Title "BeagleDust Leash PCB"
-Date "2019-07-22"
-Rev "1"
+Date "2019-08-12"
+Rev "A"
 Comp "Beagleboard.org"
 Comment1 "Schematic designed by Analog Life, LLC"
@@
 F 7 "S2B-PH-SM4-TB(LF)(SN)" H 7500 4725 50  0001 C CNN "MPN1"
 F 8 "JST Sales America Inc." H 7500 4725 50  0001 C CNN "Vendor1"
+F 9 "CONN HEADER SMD R/A 2POS 2MM" H 7500 4725 50  0001 C CNN "Short Description"
 	1    7500 4725
 	1    0    0    -1
@@
 F 7 "$0.02037" H 8750 4725 50  0001 C CNN "Standard Price"
 F 8 "Nexperia USA Inc." H 8750 4725 50  0001 C CNN "Vendor1"
+F 9 "DIODE SCHOTTKY 30V 200MA SOD123" H 8750 4725 50  0001 C CNN "Short Description"
 	1    8750 4725
 	-1   0    0    1

Commit message: Migrated all hierarchical labels to global labels
Changed lines of the file:
@@
 Wire Wire Line
 	8900 4725 9600 4725
-Text HLabel 9600 4725 2    118  Input ~ 0
-V_ALT
 Text Label 8200 4725 0    50   ~ 0
 ALT_IN
@@
 Wire Wire Line
 	7700 4725 8600 4725
+Text GLabel 9600 4725 2    63   Input ~ 0
+V_ALT
 $EndSCHEMATC

Commit message: Removed two extra pullup resistors
Parts:
- renumbered D301 to D201, J301 to J201
Changed lines of the file:
@@
 P 7500 4725
 AR Path="/5D080251" Ref="J?"  Part="1"
-AR Path="/5D0603E8/5D080251" Ref="J301"  Part="1"
-F 0 "J301" H 7608 4906 50  0000 C CNN
+AR Path="/5D0603E8/5D080251" Ref="J201"  Part="1"
+F 0 "J201" H 7608 4906 50  0000 C CNN
 F 1 "Conn_01x02_Male" H 7608 4815 50  0000 C CNN
 F 2 "Connector_JST:JST_PH_S2B-PH-SM4-TB_1x02-1MP_P2.00mm_Horizontal" H 7500 4725 50  0001 C CNN
@@
 P 8000 5175
 AR Path="/5D080259" Ref="#PWR?"  Part="1"
-AR Path="/5D0603E8/5D080259" Ref="#PWR0301"  Part="1"
-F 0 "#PWR0301" H 8000 4925 50  0001 C CNN
+AR Path="/5D0603E8/5D080259" Ref="#PWR0201"  Part="1"
+F 0 "#PWR0201" H 8000 4925 50  0001 C CNN
 F 1 "GND" H 8005 5002 50  0000 C CNN
 F 2 "" H 8000 5175 50  0001 C CNN
@@
 ALT_IN
 $Comp
-L Device:D_Schottky D301
+L Device:D_Schottky D201
 U 1 1 5D0807BE
 P 8750 4725
-F 0 "D301" H 8750 4500 50  0000 C CNN
+F 0 "D201" H 8750 4500 50  0000 C CNN
 F 1 "BAT54" H 8750 4591 50  0000 C CNN
 F 2 "Diode_SMD:D_SOD-123" H 8750 4550 50  0001 C CNN

Commit message: Added new components and hooked MSP430 into the SPI flash and the lines for programming the CC1352
Connections:
- wire segments 4 -> 7
Changed lines of the file:
@@
 Wire Wire Line
 	8900 4725 9600 4725
-Text Label 8200 4725 0    50   ~ 0
-ALT_IN
 $Comp
 L Device:D_Schottky D201
@@
 No pop if using the \nswitch/jumper method
 Wire Wire Line
-	7700 4725 8600 4725
+	7700 4725 8325 4725
 Text GLabel 9600 4725 2    63   Input ~ 0
 V_ALT
+Text GLabel 8575 4300 2    63   Input ~ 0
+ALT_IN
+Wire Wire Line
+	8575 4300 8325 4300
+Wire Wire Line
+	8325 4300 8325 4725
+Connection ~ 8325 4725
+Wire Wire Line
+	8325 4725 8600 4725
 $EndSCHEMATC

Commit message: Updated BOM for ordering parts
Parts:
- J201: Link1 https://www.digikey.com/product-detail/en/jst-sales-america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 -> https://SeeedStudio.com; Link2 (none) -> https://www.digikey.com/product-detail/en/jst-sales-america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; MPN1 S2B-PH-SM4-TB(LF)(SN) -> A2001WF-02A; MPN2 (none) -> S2B-PH-SM4-TB(LF)(SN); Vendor1 JST Sales America Inc. -> Seeed Studio; Vendor2 (none) -> JST Sales America Inc.
Changed lines of the file:
@@
 F 3 "~" H 7500 4725 50  0001 C CNN
 F 4 "$0.03" H 7500 4725 50  0001 C CNN "Standard Price"
-F 5 "https://www.digikey.com/product-detail/en/jst-sales-america-inc/S2B-PH-SM4-TB-LF-SN/455-1749-1-ND/926846" H 7500 4725 50  0001 C CNN "Link1"
+F 5 "https://SeeedStudio.com" H 7500 4725 50  0001 C CNN "Link1"
 F 6 "CONN HEADER SMD R/A 2POS 2MM" H 7500 4725 50  0001 C CNN "Description"
-F 7 "S2B-PH-SM4-TB(LF)(SN)" H 7500 4725 50  0001 C CNN "MPN1"
-F 8 "JST Sales America Inc." H 7500 4725 50  0001 C CNN "Vendor1"
+F 7 "A2001WF-02A" H 7500 4725 50  0001 C CNN "MPN1"
+F 8 "Seeed Studio" H 7500 4725 50  0001 C CNN "Vendor1"
 F 9 "CONN HEADER SMD R/A 2POS 2MM" H 7500 4725 50  0001 C CNN "Short Description"
+F 10 "https://www.digikey.com/product-detail/en/jst-sales-america-inc/S2B-PH-SM4-TB-LF-SN/455-1749-1-ND/926846" H 7500 4725 50  0001 C CNN "Link2"
+F 11 "S2B-PH-SM4-TB(LF)(SN)" H 7500 4725 50  0001 C CNN "MPN2"
+F 12 "JST Sales America Inc." H 7500 4725 50  0001 C CNN "Vendor2"
 	1    7500 4725
 	1    0    0    -1
