File: hw/LeashPCB/Sensors.sch (KiCad schematic (older format))
At the start: 13 parts, among them U1001 HDC2010, U1002 SN74AUP2G32, U1003 LTR-303ALS-01, U1004 LIS2DE12

Commit message: Added new components and hooked MSP430 into the SPI flash and the lines for programming the CC1352
Parts:
- added R1008: 0, Resistor_SMD:R_0402_1005Metric, symbol Device:R
- U1003: value LTR-303ALS-01 -> OPT3001; footprint OptoDevice:Lite-On_LTR-303ALS-01 -> leash:USON6; symbol Sensor_Optical:LTR-303ALS-01 -> LeashPCB:OPT3001; Link1 (none) -> http://www.ti.com/product/OPT3001/samplebuy; MPN1 (none) -> OPT3001DNPR; Standard Price (none) -> 0.2175
Connections:
- net labels added: INT_OPT3001
- net labels removed: INT_LTR303
- wire segments 67 -> 70
Changed lines of the file:
@@
 $EndComp
 $Comp
-L Sensor_Optical:LTR-303ALS-01 U1003
+L LeashPCB:OPT3001 U1003
 U 1 1 5E7503C1
 P 2775 5725
 F 0 "U1003" H 2475 6075 50  0000 L CNN
-F 1 "LTR-303ALS-01" H 2825 6075 50  0000 L CNN
-F 2 "OptoDevice:Lite-On_LTR-303ALS-01" H 2775 6175 50  0001 C CNN
-F 3 "http://optoelectronics.liteon.com/upload/download/DS86-2013-0004/LTR-303ALS-01_DS_V1.pdf" H 2475 6075 50  0001 C CNN
+F 1 "OPT3001" H 2825 6075 50  0000 L CNN
+F 2 "leash:USON6" H 2775 6175 50  0001 C CNN
+F 3 "http://www.ti.com/lit/ds/symlink/opt3001.pdf" H 2475 6075 50  0001 C CNN
+F 4 "OPT3001DNPR" H 2775 5725 50  0001 C CNN "MPN1"
+F 5 "0.2175" H 2775 5725 50  0001 C CNN "Standard Price"
+F 6 "http://www.ti.com/product/OPT3001/samplebuy" H 2775 5725 50  0001 C CNN "Link1"
 	1    2775 5725
 	1    0    0    -1
@@
 Wire Wire Line
 	2775 6125 2775 6275
-Text GLabel 7700 2750 0    50   Input ~ 0
-INT_LTR303
-Text GLabel 3350 5725 2    50   Input ~ 0
-INT_LTR303
-Wire Wire Line
-	3350 5725 3175 5725
+Text GLabel 3350 5625 2    50   Input ~ 0
+INT_OPT3001
+Wire Wire Line
+	3350 5625 3175 5625
 Text GLabel 5025 5725 0    50   Input ~ 0
 SCL
@@
 Text GLabel 4475 3300 0    50   Input ~ 0
 INT_HDC2010
+$Comp
+L Device:R R?
+U 1 1 5E4E359C
+P 3475 5825
+AR Path="/5D062750/5E4E359C" Ref="R?"  Part="1"
+AR Path="/5E6C68DD/5E4E359C" Ref="R1008"  Part="1"
+F 0 "R1008" V 3425 5600 50  0000 L CNN
+F 1 "0" V 3475 5800 50  0000 L CNN
+F 2 "Resistor_SMD:R_0402_1005Metric" V 3405 5825 50  0001 C CNN
+F 3 "~" H 3475 5825 50  0001 C CNN
+F 4 "RES 0 OHM JUMPER 1/16W 0402" H 3475 5825 50  0001 C CNN "Description"
+F 5 "https://www.digikey.com/product-detail/en/stackpole-electronics-inc/RMCF0402ZT0R00/RMCF0402ZT0R00TR-ND/1756905" H 3475 5825 50  0001 C CNN "Link1"
+F 6 "RMCF0402ZT0R00" H 3475 5825 50  0001 C CNN "MPN1"
+F 7 "$0.00127" H 3475 5825 50  0001 C CNN "Standard Price"
+F 8 "Stackpole Electronics Inc" H 3475 5825 50  0001 C CNN "Vendor1"
+F 9 "RES 0 OHM JUMPER 1/16W 0402" H 3475 5825 50  0001 C CNN "Short Description"
+	1    3475 5825
+	0    1    1    0
+$EndComp
+Wire Wire Line
+	3175 5825 3325 5825
+Wire Wire Line
+	3700 5825 3700 6125
+Wire Wire Line
+	3625 5825 3700 5825
+$Comp
+L power:GND #PWR0110
+U 1 1 5E4E591F
+P 3700 6125
+F 0 "#PWR0110" H 3700 5875 50  0001 C CNN
+F 1 "GND" H 3700 5975 50  0000 C CNN
+F 2 "" H 3700 6125 50  0001 C CNN
+F 3 "" H 3700 6125 50  0001 C CNN
+	1    3700 6125
+	1    0    0    -1
+$EndComp
+Text GLabel 7700 2750 0    50   Input ~ 0
+INT_OPT3001
 $EndSCHEMATC

Commit message: Updated BOM for ordering parts
Parts:
- R1001, R1002: Standard Price $0.00563 -> 0.00498
- U1001: Link1 http://www.ti.com/product/HDC2010 -> https://www.digikey.com/product-detail/en/texas-instruments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; MPN1 (none) -> HDC2010YPAR; Short Description (none) -> GEN 2 HUMIDITY SENSOR; Standard Price (none) -> 0.2175; Vendor1 (none) -> Texas Instruments
- U1002: Link1 (none) -> https://www.digikey.com/product-detail/en/texas-instruments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; MPN1 (none) -> SN74AUP2G32DQER; Short Description (none) -> IC GATE OR 2CH 2-INP 8X2SON; Standard Price (none) -> 0.0225; Vendor1 (none) -> Texas Instruments
- U1003: Link1 http://www.ti.com/product/OPT3001/samplebuy -> https://www.digikey.com/product-detail/en/texas-instruments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; Short Description (none) -> SENSOR OPT 550NM AMBIENT 6USON; Vendor1 (none) -> Texas Instruments
- U1004: Link1 (none) -> https://www.digikey.com/products/en/sensors-transducers/mot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; MPN1 (none) -> LIS2DE12TR; Short Description (none) -> ACCEL 2-16G I2C/SPI 12LGA; Standard Price (none) -> 0.51200; Vendor1 (none) -> STMicroelectronics
Changed lines of the file:
@@
 F 2 "leash:HDC2010" H 5425 3400 50  0001 C CNN
 F 3 "http://www.ti.com/lit/ds/symlink/hdc2010.pdf" H 5425 3400 50  0001 C CNN
-F 4 "http://www.ti.com/product/HDC2010" H 5425 3250 50  0001 C CNN "Link1"
+F 4 "https://www.digikey.com/product-detail/en/texas-instruments/HDC2010YPAR/296-47774-2-ND/7561364" H 5425 3250 50  0001 C CNN "Link1"
+F 5 "HDC2010YPAR" H 5425 3250 50  0001 C CNN "MPN1"
+F 6 "GEN 2 HUMIDITY SENSOR" H 5425 3250 50  0001 C CNN "Short Description"
+F 7 "0.2175" H 5425 3250 50  0001 C CNN "Standard Price"
+F 8 "Texas Instruments" H 5425 3250 50  0001 C CNN "Vendor1"
 	1    5425 3250
 	1    0    0    -1
@@
 F 5 "https://www.digikey.com/product-detail/en/panasonic-electronic-components/ERJ-2RKF2211X/P2.21KLTR-ND/192198" H 4550 2500 50  0001 C CNN "Link1"
 F 6 "ERJ-2RKF2211X" H 4550 2500 50  0001 C CNN "MPN1"
-F 7 "$0.00563	" H 4550 2500 50  0001 C CNN "Standard Price"
+F 7 "0.00498" H 4550 2500 50  0001 C CNN "Standard Price"
 F 8 "Panasonic Electronic Components" H 4550 2500 50  0001 C CNN "Vendor1"
 F 9 "RES SMD 2.21K OHM 1% 1/10W 0402" H 4550 2500 50  0001 C CNN "Short Description"
@@
 F 5 "https://www.digikey.com/product-detail/en/panasonic-electronic-components/ERJ-2RKF2211X/P2.21KLTR-ND/192198" H 4900 2500 50  0001 C CNN "Link1"
 F 6 "ERJ-2RKF2211X" H 4900 2500 50  0001 C CNN "MPN1"
-F 7 "$0.00563	" H 4900 2500 50  0001 C CNN "Standard Price"
+F 7 "0.00498" H 4900 2500 50  0001 C CNN "Standard Price"
 F 8 "Panasonic Electronic Components" H 4900 2500 50  0001 C CNN "Vendor1"
 F 9 "RES SMD 2.21K OHM 1% 1/10W 0402" H 4900 2500 50  0001 C CNN "Short Description"
@@
 F 2 "Package_SON:X2SON-8_1.4x1mm_P0.35mm" H 8725 2900 50  0001 C CNN
 F 3 "http://www.ti.com/lit/ds/symlink/sn74aup2g32.pdf" H 8725 2900 50  0001 C CNN
+F 4 "https://www.digikey.com/product-detail/en/texas-instruments/SN74AUP2G32DQER/296-25873-2-ND/2242310" H 8825 2800 50  0001 C CNN "Link1"
+F 5 "SN74AUP2G32DQER" H 8825 2800 50  0001 C CNN "MPN1"
+F 6 "IC GATE OR 2CH 2-INP 8X2SON" H 8825 2800 50  0001 C CNN "Short Description"
+F 7 "0.0225" H 8825 2800 50  0001 C CNN "Standard Price"
+F 8 "Texas Instruments" H 8825 2800 50  0001 C CNN "Vendor1"
 	1    8825 2800
 	1    0    0    -1
@@
 F 2 "Package_LGA:LGA-12_2x2mm_P0.5mm" H 6300 6175 50  0001 L CNN
 F 3 "https://www.st.com/resource/en/datasheet/lis2DE12.pdf" H 5800 5625 50  0001 C CNN
+F 4 "https://www.digikey.com/products/en/sensors-transducers/motion-sensors-accelerometers/515?k=LIS2DE12&k=&pkeyword=LIS2DE12&sv=0&pv7=1&sf=0&FV=-8%7C515&quantity=&ColumnSort=0&page=1&pageSize=25" H 6150 5625 50  0001 C CNN "Link1"
+F 5 "LIS2DE12TR" H 6150 5625 50  0001 C CNN "MPN1"
+F 6 "ACCEL 2-16G I2C/SPI 12LGA" H 6150 5625 50  0001 C CNN "Short Description"
+F 7 "0.51200" H 6150 5625 50  0001 C CNN "Standard Price"
+F 8 "STMicroelectronics" H 6150 5625 50  0001 C CNN "Vendor1"
 	1    6150 5625
 	1    0    0    -1
@@
 F 4 "OPT3001DNPR" H 2775 5725 50  0001 C CNN "MPN1"
 F 5 "0.2175" H 2775 5725 50  0001 C CNN "Standard Price"
-F 6 "http://www.ti.com/product/OPT3001/samplebuy" H 2775 5725 50  0001 C CNN "Link1"
+F 6 "https://www.digikey.com/product-detail/en/texas-instruments/OPT3001DNPR/296-40474-2-ND/5039362" H 2775 5725 50  0001 C CNN "Link1"
+F 7 "SENSOR OPT 550NM AMBIENT 6USON" H 2775 5725 50  0001 C CNN "Short Description"
+F 8 "Texas Instruments" H 2775 5725 50  0001 C CNN "Vendor1"
 	1    2775 5725
 	1    0    0    -1

Commit message: Revisions and fixes for Rev B board in preparation for Rev C start. Changed how we handle the MSP430 and how it connects to the cc1352r. Also some part swaps and pin swaps on the cc1352r. Fixes #4 and #5.
Parts:
- C1001, C1002: value 0.1 uF -> 0.1U
- R1007: value 0 -> 2.21K; Description RES 0 OHM JUMPER 1/16W 0402 -> RES SMD 2.21K OHM 1% 1/10W 0402; Link1 https://www.digikey.com/product-detail/en/stackpole-electro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 -> https://www.digikey.com/product-detail/en/panasonic-electro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; MPN1 RMCF0402ZT0R00 -> ERJ-2RKF2211X; Short Description RES 0 OHM JUMPER 1/16W 0402 -> RES SMD 2.21K OHM 1% 1/10W 0402; Standard Price $0.00127 -> 0.00498; Vendor1 Stackpole Electronics Inc -> Panasonic Electronic Components
Connections:
- net labels added: INT_MB2
- net labels removed: INT_LIS2DE12, INT_OPT3001
Changed lines of the file:
@@
 AR Path="/5E6C68DD/5E6D759A" Ref="C1001"  Part="1"
 F 0 "C1001" H 3135 2379 50  0000 R CNN
-F 1 "0.1 uF" H 3135 2470 50  0000 R CNN
+F 1 "0.1U" H 3135 2470 50  0000 R CNN
 F 2 "Capacitor_SMD:C_0402_1005Metric" H 3288 2275 50  0001 C CNN
 F 3 "~" H 3250 2425 50  0001 C CNN
@@
 AR Path="/5E6C68DD/5E6E5EA9" Ref="C1002"  Part="1"
 F 0 "C1002" H 10310 2879 50  0000 R CNN
-F 1 "0.1 uF" H 10310 2970 50  0000 R CNN
+F 1 "0.1U" H 10310 2970 50  0000 R CNN
 F 2 "Capacitor_SMD:C_0402_1005Metric" H 10463 2775 50  0001 C CNN
 F 3 "~" H 10425 2925 50  0001 C CNN
@@
 INT_SENSOR
 Wire Wire Line
-	8425 2750 8200 2750
-Wire Wire Line
 	9425 3050 9225 3050
 $Comp
@@
 	2775 5100 2775 5325
 Wire Wire Line
-	5650 4725 6150 4725
+	4875 4725 5250 4725
 Wire Wire Line
 	6150 4725 6150 5125
@@
 Wire Wire Line
 	2775 6125 2775 6275
-Text GLabel 3350 5625 2    50   Input ~ 0
-INT_OPT3001
 Wire Wire Line
 	3350 5625 3175 5625
@@
 Wire Wire Line
 	6975 5525 6650 5525
-Text GLabel 9425 3050 2    50   Input ~ 0
-INT_LIS2DE12
 Wire Wire Line
 	6650 5925 6775 5925
@@
 Wire Wire Line
 	6975 5625 6650 5625
-Text GLabel 7675 2625 0    50   Input ~ 0
+Text GLabel 8050 2750 0    50   Input ~ 0
 INT_LIS2DE12_2
 Wire Wire Line
@@
 Wire Wire Line
 	8000 2225 8300 2225
-$Comp
-L Device:R R?
-U 1 1 5E78AEF0
-P 7950 2750
-AR Path="/5D062750/5E78AEF0" Ref="R?"  Part="1"
-AR Path="/5E6C68DD/5E78AEF0" Ref="R1007"  Part="1"
-F 0 "R1007" V 7900 2525 50  0000 L CNN
-F 1 "0" V 7950 2725 50  0000 L CNN
-F 2 "Resistor_SMD:R_0402_1005Metric" V 7880 2750 50  0001 C CNN
-F 3 "~" H 7950 2750 50  0001 C CNN
-F 4 "RES 0 OHM JUMPER 1/16W 0402" H 7950 2750 50  0001 C CNN "Description"
-F 5 "https://www.digikey.com/product-detail/en/stackpole-electronics-inc/RMCF0402ZT0R00/RMCF0402ZT0R00TR-ND/1756905" H 7950 2750 50  0001 C CNN "Link1"
-F 6 "RMCF0402ZT0R00" H 7950 2750 50  0001 C CNN "MPN1"
-F 7 "$0.00127" H 7950 2750 50  0001 C CNN "Standard Price"
-F 8 "Stackpole Electronics Inc" H 7950 2750 50  0001 C CNN "Vendor1"
-F 9 "RES 0 OHM JUMPER 1/16W 0402" H 7950 2750 50  0001 C CNN "Short Description"
-	1    7950 2750
-	0    -1   -1   0
-$EndComp
-Wire Wire Line
-	7800 2750 7700 2750
-$Comp
-L Device:R R?
-U 1 1 5E78B7F5
-P 7950 2625
-AR Path="/5D062750/5E78B7F5" Ref="R?"  Part="1"
-AR Path="/5E6C68DD/5E78B7F5" Ref="R1006"  Part="1"
-F 0 "R1006" V 7900 2400 50  0000 L CNN
-F 1 "0" V 7950 2600 50  0000 L CNN
-F 2 "Resistor_SMD:R_0402_1005Metric" V 7880 2625 50  0001 C CNN
-F 3 "~" H 7950 2625 50  0001 C CNN
-F 4 "RES 0 OHM JUMPER 1/16W 0402" H 7950 2625 50  0001 C CNN "Description"
-F 5 "https://www.digikey.com/product-detail/en/stackpole-electronics-inc/RMCF0402ZT0R00/RMCF0402ZT0R00TR-ND/1756905" H 7950 2625 50  0001 C CNN "Link1"
-F 6 "RMCF0402ZT0R00" H 7950 2625 50  0001 C CNN "MPN1"
-F 7 "$0.00127" H 7950 2625 50  0001 C CNN "Standard Price"
-F 8 "Stackpole Electronics Inc" H 7950 2625 50  0001 C CNN "Vendor1"
-F 9 "RES 0 OHM JUMPER 1/16W 0402" H 7950 2625 50  0001 C CNN "Short Description"
-F 10 "DNP" V 7975 2425 50  0000 C CNN "Population"
-	1    7950 2625
-	0    -1   -1   0
-$EndComp
-Wire Wire Line
-	8100 2625 8200 2625
-Wire Wire Line
-	8200 2625 8200 2750
-Connection ~ 8200 2750
-Wire Wire Line
-	8200 2750 8100 2750
-Wire Wire Line
-	7800 2625 7675 2625
-Text GLabel 5650 4725 0    50   Input ~ 0
+Text GLabel 4875 4725 0    50   Input ~ 0
 VDDS
 Text GLabel 3200 2100 0    50   Input ~ 0
@@
 AR Path="/5D062750/5E4E359C" Ref="R?"  Part="1"
 AR Path="/5E6C68DD/5E4E359C" Ref="R1008"  Part="1"
-F 0 "R1008" V 3425 5600 50  0000 L CNN
+F 0 "R1008" V 3550 5500 50  0000 L CNN
 F 1 "0" V 3475 5800 50  0000 L CNN
 F 2 "Resistor_SMD:R_0402_1005Metric" V 3405 5825 50  0001 C CNN
@@
 	1    0    0    -1
 $EndComp
-Text GLabel 7700 2750 0    50   Input ~ 0
-INT_OPT3001
+Wire Wire Line
+	8050 2750 8425 2750
+$Comp
+L Device:R R?
+U 1 1 5F5F1CFB
+P 3500 5625
+AR Path="/5D062750/5F5F1CFB" Ref="R?"  Part="1"
+AR Path="/5E6C68DD/5F5F1CFB" Ref="R1006"  Part="1"
+F 0 "R1006" V 3450 5275 50  0000 L CNN
+F 1 "0" V 3500 5600 50  0000 L CNN
+F 2 "Resistor_SMD:R_0402_1005Metric" V 3430 5625 50  0001 C CNN
+F 3 "~" H 3500 5625 50  0001 C CNN
+F 4 "RES 0 OHM JUMPER 1/16W 0402" H 3500 5625 50  0001 C CNN "Description"
+F 5 "https://www.digikey.com/product-detail/en/stackpole-electronics-inc/RMCF0402ZT0R00/RMCF0402ZT0R00TR-ND/1756905" H 3500 5625 50  0001 C CNN "Link1"
+F 6 "RMCF0402ZT0R00" H 3500 5625 50  0001 C CNN "MPN1"
+F 7 "$0.00127" H 3500 5625 50  0001 C CNN "Standard Price"
+F 8 "Stackpole Electronics Inc" H 3500 5625 50  0001 C CNN "Vendor1"
+F 9 "RES 0 OHM JUMPER 1/16W 0402" H 3500 5625 50  0001 C CNN "Short Description"
+F 10 "DNP" V 3550 5450 50  0000 C CNN "Population"
+	1    3500 5625
+	0    -1   -1   0
+$EndComp
+Wire Wire Line
+	3650 5625 4050 5625
+Text GLabel 4050 5625 2    50   Input ~ 0
+INT_MB2
+$Comp
+L Device:R R?
+U 1 1 5F5FF654
+P 5250 5125
+AR Path="/5D062750/5F5FF654" Ref="R?"  Part="1"
+AR Path="/5E6C68DD/5F5FF654" Ref="R1007"  Part="1"
+F 0 "R1007" H 5320 5171 50  0000 L CNN
+F 1 "2.21K" H 5320 5080 50  0000 L CNN
+F 2 "Resistor_SMD:R_0402_1005Metric" V 5180 5125 50  0001 C CNN
+F 3 "~" H 5250 5125 50  0001 C CNN
+F 4 "RES SMD 2.21K OHM 1% 1/10W 0402" H 5250 5125 50  0001 C CNN "Description"
+F 5 "https://www.digikey.com/product-detail/en/panasonic-electronic-components/ERJ-2RKF2211X/P2.21KLTR-ND/192198" H 5250 5125 50  0001 C CNN "Link1"
+F 6 "ERJ-2RKF2211X" H 5250 5125 50  0001 C CNN "MPN1"
+F 7 "0.00498" H 5250 5125 50  0001 C CNN "Standard Price"
+F 8 "Panasonic Electronic Components" H 5250 5125 50  0001 C CNN "Vendor1"
+F 9 "RES SMD 2.21K OHM 1% 1/10W 0402" H 5250 5125 50  0001 C CNN "Short Description"
+	1    5250 5125
+	1    0    0    -1
+$EndComp
+Wire Wire Line
+	5750 5425 5250 5425
+Wire Wire Line
+	5250 5425 5250 5275
+Wire Wire Line
+	5250 4975 5250 4725
+Connection ~ 5250 4725
+Wire Wire Line
+	5250 4725 6150 4725
+Text GLabel 9425 3050 2    50   Input ~ 0
+INT_LIS2DE12_1
 $EndSCHEMATC
