File: hw/LeashPCB/Sensors.sch (KiCad schematic (older format))
At the start: 14 parts, among them U1001 HDC2010, U1002 SN74AUP2G32, U1003 OPT3001, U1004 LIS2DE12

Commit message: Schematic update by seeed
1. BOM match seeed components library
2. Modify U1 VBUS pin connection
3. Add 100nF decoupling capacitor for sensors
Parts:
- added C41, C42: 0.1U, Capacitor_SMD:C_0402_1005Metric, symbol Device:C
- C40: renamed from C1001; MPN2 (none) -> CC0402KRX5R6BB104; Seeed Description (none) -> SMD CAP Ceramic 100nF-10V-10%-X5R;0402; Seeed PN (none) -> 302011121; Vendor2 (none) -> YAGEO
- C43: renamed from C1002; MPN2 (none) -> CC0402KRX5R6BB104; Seeed Description (none) -> SMD CAP Ceramic 100nF-10V-10%-X5R;0402; Seeed PN (none) -> 302011121; Vendor2 (none) -> YAGEO
- R48: renamed from R1008; MPN2 (none) -> RC0402JR-070RL; Seeed Description (none) -> SMD RES 0R-5%-1/16W;0402; Seeed PN (none) -> 301010000; Vendor2 (none) -> YAGEO
- R49: renamed from R1006; MPN2 (none) -> RC0402JR-070RL; Seeed Description (none) -> SMD RES 0R-5%-1/16W;0402; Seeed PN (none) -> 301010000; Vendor2 (none) -> YAGEO
- R50: renamed from R1001; MPN2 (none) -> RC0402FR-072K21L; Seeed Description (none) -> SMD RES 2.21K-1%-1/16W;0402; Seeed PN (none) -> 301010881; Vendor2 (none) -> YAGEO
- R51: renamed from R1004; MPN2 (none) -> RC0402JR-070RL; Seeed Description (none) -> SMD RES 0R-5%-1/16W;0402; Seeed PN (none) -> 301010000; Vendor2 (none) -> YAGEO
- R52: renamed from R1002; MPN2 (none) -> RC0402FR-072K21L; Seeed Description (none) -> SMD RES 2.21K-1%-1/16W;0402; Seeed PN (none) -> 301010881; Vendor2 (none) -> YAGEO
- R53: renamed from R1007; MPN2 (none) -> RC0402FR-072K21L; Seeed Description (none) -> SMD RES 2.21K-1%-1/16W;0402; Seeed PN (none) -> 301010881; Vendor2 (none) -> YAGEO
- R54: renamed from R1005; MPN2 (none) -> RC0402JR-070RL; Seeed Description (none) -> SMD RES 0R-5%-1/16W;0402; Seeed PN (none) -> 301010000; Vendor2 (none) -> YAGEO
- R55: renamed from R1003; MPN2 (none) -> RC0402JR-070RL; Seeed Description (none) -> SMD RES 0R-5%-1/16W;0402; Seeed PN (none) -> 301010000; Vendor2 (none) -> YAGEO
- U10: renamed from U1002; symbol LeashPCB:SN74AUP2G32 -> LeashPCB:SN74AUP2G32-LeashPCB; Seeed PN (none) -> 0
- U7: renamed from U1003; symbol LeashPCB:OPT3001 -> LeashPCB:OPT3001-LeashPCB; MPN2 (none) -> OPT3001DNPR; Seeed Description (none) -> SMD Optical Sensor;UDFN-6; Seeed PN (none) -> 314020321; Vendor2 (none) -> TI
- U8: renamed from U1001; symbol LeashPCB:HDC2010 -> LeashPCB:HDC2010-LeashPCB; Seeed PN (none) -> 0
- U9: renamed from U1004; symbol Sensor_Motion:LIS2DE12 -> LeashPCB:LIS2DE12-lis2hh12; MPN2 (none) -> LIS2DE12TR; Seeed Description (none) -> （Fusion）SMD Motion & Position Sensor;LGA-12; Seeed PN (none) -> 314080306; Vendor2 (none) -> ST
Connections:
- net labels added: 3V3
- net labels removed: VDDS
- wire segments 70 -> 76
Other:
- moved on the sheet: C40
