File: hw/LeashPCB/Boost.sch (KiCad schematic (older format))
At the start: 44 parts, among them SW801 SW_SPDT, U1001 TPS62821DLC, U1002 TPS61026, U1003 TPS61025

Commit message: Swapped out USB and antenna sections and refactored outline, started routing
Parts:
- removed C1001, C1002, C1006, C1008: 10 uF, Capacitor_SMD:C_0402_1005Metric, symbol Device:C
- removed C1004, C1005: 2.2 uF, Capacitor_SMD:C_0402_1005Metric, symbol Device:C
- removed JP801, JP802, JP803, JP804, JP805: SolderJumper_2_Bridged, Jumper:SolderJumper-2_P1.3mm_Bridged2Bar_RoundedPad1.0x1.5mm, symbol Jumper:SolderJumper_2_Bridged
- removed L1001, L1002: 6.8 uH, leash:CDRH4D28, symbol pspice:INDUCTOR
- removed R10, R1006, R1017, R1018, R801, R802, R803, R804, R9: 0, Resistor_SMD:R_0402_1005Metric, symbol Device:R
- removed R1002, R1004: 200K, Resistor_SMD:R_0402_1005Metric, symbol Device:R
- removed R1003, R1005: 390K, Resistor_SMD:R_0402_1005Metric, symbol Device:R
- removed R1007, R1009, R1010, R1011, R1012: 10K, Resistor_SMD:R_0402_1005Metric, symbol Device:R
- removed R1013, R1016: 1 MEG, Resistor_SMD:R_0402_1005Metric, symbol Device:R
- removed SW801: SW_SPDT, leash:K3-1293S-E2, symbol Switch:SW_SPDT
- removed U1002: TPS61026, Package_SON:VSON-10-1EP_3x3mm_P0.5mm_EP1.65x2.4mm_ThermalVias, symbol LeashPCB:TPS61026
- removed U1003: TPS61025, Package_SON:VSON-10-1EP_3x3mm_P0.5mm_EP1.65x2.4mm_ThermalVias, symbol LeashPCB:TPS61025
- added R708: 0, Resistor_SMD:R_0402_1005Metric, symbol Device:R
Connections:
- net labels added: 3V3_BUCK_IN
- net labels removed: +5V, 3V3_BOOST_VIN, 3V3_BOOST_VOUT, 3v3_CTRL, 5V_BOOST_VIN, 5V_BOOST_VOUT, 5V_CTRL, 5V_EN, 5V_REG, V_BAT
- wire segments 187 -> 42
Other:
- note removed: "Adding in a low cost, small switch for\nfuture cost reduction. Removes the need\nfor ideal diode controller."
- note removed: "CONFIG 1: All power inputs go into 3V3 boost, ALT and USB go into the 5V boost\nCONFIG 2: All power inputs go into 3V3 boost, all go into the 5V boost\nCONFIG 3: All power inputs go into 5V boost, 5V is bucked down to 3V3\nCONFIG 4: User has to manually swich from internal power to external power, which are diode ORed together"
- note removed: "Not normally populated"
- note removed: "Optional pull up resistor\nto change to default on \nbehavior"
- note removed: "V_Bat not hooked into \n5V output normally"
- moved on the sheet: C1003, C1007, C1009, L1003, R1008, R1014, R1015

Commit message: Migrated all hierarchical labels to global labels
Connections:
- net labels added: 3V3
- net labels removed: +3V3, 3V3_REG
- wire segments 42 -> 41
Changed lines of the file:
@@
 $Descr B 17000 11000
 encoding utf-8
-Sheet 7 9
+Sheet 6 9
 Title "BeagleDust Leash PCB"
 Date "2019-08-12"
@@
 	8550 5725 8550 5625
 $Comp
-L power:GND #PWR0128
-U 1 1 5D20C65C
-P 8275 8450
-F 0 "#PWR0128" H 8275 8200 50  0001 C CNN
-F 1 "GND" H 8280 8277 50  0000 C CNN
-F 2 "" H 8275 8450 50  0001 C CNN
-F 3 "" H 8275 8450 50  0001 C CNN
-	1    8275 8450
-	1    0    0    -1
-$EndComp
-$Comp
 L Device:C C1009
 U 1 1 5D20CB94
@@
 Connection ~ 6850 5075
 Wire Wire Line
-	6850 5075 7450 5075
+	6850 5075 7100 5075
 Wire Wire Line
 	6275 5075 6275 5175
@@
 Wire Wire Line
 	5325 5075 6275 5075
-Text HLabel 14150 4600 2    118  Input ~ 0
-3V3_REG
 Text Label 10850 5075 0    50   ~ 0
 3V3_BUCK_VOUT
-$Comp
-L power:+3V3 #PWR0150
-U 1 1 5D3B8759
-P 13800 4425
-F 0 "#PWR0150" H 13800 4275 50  0001 C CNN
-F 1 "+3V3" H 13815 4598 50  0000 C CNN
-F 2 "" H 13800 4425 50  0001 C CNN
-F 3 "" H 13800 4425 50  0001 C CNN
-	1    13800 4425
-	1    0    0    -1
-$EndComp
-Wire Wire Line
-	13800 4425 13800 4600
-Wire Wire Line
-	13800 4600 14150 4600
 Wire Wire Line
 	9825 5075 10350 5075
@@
 	0    1    1    0
 $EndComp
-Wire Wire Line
-	12450 5075 13800 5075
-Wire Wire Line
-	13800 5075 13800 4600
-Connection ~ 13800 4600
 Text Label 5575 5075 0    79   ~ 0
 3V3_BUCK_IN
-Text HLabel 3225 4300 0    79   Input ~ 0
-V_USB
-Text HLabel 3225 6150 0    79   Input ~ 0
-V_ALT
 Wire Wire Line
 	3225 6150 5325 6150
@@
 	5325 4300 5325 5075
 Connection ~ 5325 5075
+Wire Wire Line
+	12450 5075 12875 5075
+Text GLabel 12875 5075 2    63   Input ~ 0
+3V3
+$Comp
+L power:GND #PWR0122
+U 1 1 5E9441DB
+P 9825 6025
+F 0 "#PWR0122" H 9825 5775 50  0001 C CNN
+F 1 "GND" H 9830 5852 50  0000 C CNN
+F 2 "" H 9825 6025 50  0001 C CNN
+F 3 "" H 9825 6025 50  0001 C CNN
+	1    9825 6025
+	1    0    0    -1
+$EndComp
+Text GLabel 3225 4300 0    63   Input ~ 0
+V_USB
+Text GLabel 3225 6150 0    63   Input ~ 0
+V_ALT
+$Comp
+L power:PWR_FLAG #FLG0104
+U 1 1 5E9CDAED
+P 7100 4975
+F 0 "#FLG0104" H 7100 5050 50  0001 C CNN
+F 1 "PWR_FLAG" H 7100 5125 50  0000 C CNN
+F 2 "" H 7100 4975 50  0001 C CNN
+F 3 "~" H 7100 4975 50  0001 C CNN
+	1    7100 4975
+	1    0    0    -1
+$EndComp
+Wire Wire Line
+	7100 4975 7100 5075
+Connection ~ 7100 5075
+Wire Wire Line
+	7100 5075 7450 5075
 $EndSCHEMATC

Commit message: Removed two extra pullup resistors
Parts:
- renumbered C1003 to C601, C1007 to C602, C1009 to C603, L1003 to L601, R1008 to R601, R1014 to R602, R1015 to R603, R708 to R604, U1001 to U601
Changed lines of the file:
@@
 $EndBitmap
 $Comp
-L LeashPCB:TPS62821DLC U1001
+L LeashPCB:TPS62821DLC U601
 U 1 1 5D1D7726
 P 8025 5325
-F 0 "U1001" H 8000 5990 50  0000 C CNN
+F 0 "U601" H 8000 5990 50  0000 C CNN
 F 1 "TPS62821DLC" H 8000 5899 50  0000 C CNN
 F 2 "leash:TPS62821DLC" H 7925 5275 50  0001 C CNN
@@
 $EndComp
 $Comp
-L Device:R R1008
+L Device:R R601
 U 1 1 5D1D8A6B
 P 7200 5475
-F 0 "R1008" V 6993 5475 50  0000 C CNN
+F 0 "R601" V 6993 5475 50  0000 C CNN
 F 1 "R" V 7084 5475 50  0000 C CNN
 F 2 "Resistor_SMD:R_0402_1005Metric" V 7130 5475 50  0001 C CNN
@@
 $EndComp
 $Comp
-L pspice:INDUCTOR L1003
+L pspice:INDUCTOR L601
 U 1 1 5D1D9D03
 P 9050 5075
-F 0 "L1003" H 9050 5290 50  0000 C CNN
+F 0 "L601" H 9050 5290 50  0000 C CNN
 F 1 "INDUCTOR" H 9050 5199 50  0000 C CNN
 F 2 "leash:L_0806_2012Metric" H 9050 5075 50  0001 C CNN
@@
 $EndComp
 $Comp
-L Device:R R1014
+L Device:R R602
 U 1 1 5D1DA985
 P 9825 5275
-F 0 "R1014" H 9755 5229 50  0000 R CNN
+F 0 "R602" H 9755 5229 50  0000 R CNN
 F 1 "R" H 9755 5320 50  0000 R CNN
 F 2 "Resistor_SMD:R_0402_1005Metric" V 9755 5275 50  0001 C CNN
@@
 $EndComp
 $Comp
-L Device:R R1015
+L Device:R R603
 U 1 1 5D1DAF59
 P 9825 5675
-F 0 "R1015" H 9755 5629 50  0000 R CNN
+F 0 "R603" H 9755 5629 50  0000 R CNN
 F 1 "R" H 9755 5720 50  0000 R CNN
 F 2 "Resistor_SMD:R_0402_1005Metric" V 9755 5675 50  0001 C CNN
@@
 $EndComp
 $Comp
-L Device:C C1007
+L Device:C C602
 U 1 1 5D1DB906
 P 9525 5275
-F 0 "C1007" H 9640 5321 50  0000 L CNN
+F 0 "C602" H 9640 5321 50  0000 L CNN
 F 1 "100 pF" H 9640 5230 50  0000 L CNN
 F 2 "Capacitor_SMD:C_0402_1005Metric" H 9563 5125 50  0001 C CNN
@@
 	9525 5475 8650 5475
 $Comp
-L power:GND #PWR0127
+L power:GND #PWR0602
 U 1 1 5D204F3B
 P 8550 5850
-F 0 "#PWR0127" H 8550 5600 50  0001 C CNN
+F 0 "#PWR0602" H 8550 5600 50  0001 C CNN
 F 1 "GND" H 8555 5677 50  0000 C CNN
 F 2 "" H 8550 5850 50  0001 C CNN
@@
 	8550 5725 8550 5625
 $Comp
-L Device:C C1009
+L Device:C C603
 U 1 1 5D20CB94
 P 10350 5575
-F 0 "C1009" H 10465 5621 50  0000 L CNN
+F 0 "C603" H 10465 5621 50  0000 L CNN
 F 1 "10 uF" H 10465 5530 50  0000 L CNN
 F 2 "Capacitor_SMD:C_0603_1608Metric" H 10388 5425 50  0001 C CNN
@@
 	9825 5950 9825 6025
 $Comp
-L Device:C C1003
+L Device:C C601
 U 1 1 5D2142AD
 P 6275 5325
-F 0 "C1003" H 6390 5371 50  0000 L CNN
+F 0 "C601" H 6390 5371 50  0000 L CNN
 F 1 "1 uF" H 6390 5280 50  0000 L CNN
 F 2 "Capacitor_SMD:C_0402_1005Metric" H 6313 5175 50  0001 C CNN
@@
 	6275 5075 6850 5075
 $Comp
-L power:GND #PWR0129
+L power:GND #PWR0601
 U 1 1 5D22687F
 P 6275 5750
-F 0 "#PWR0129" H 6275 5500 50  0001 C CNN
+F 0 "#PWR0601" H 6275 5500 50  0001 C CNN
 F 1 "GND" H 6280 5577 50  0000 C CNN
 F 2 "" H 6275 5750 50  0001 C CNN
@@
 	10350 5075 12150 5075
 $Comp
-L Device:R R708
+L Device:R R604
 U 1 1 5E38DA29
 P 12300 5075
-F 0 "R708" H 12370 5166 50  0000 L CNN
+F 0 "R604" H 12370 5166 50  0000 L CNN
 F 1 "0" H 12370 5075 50  0000 L CNN
 F 2 "Resistor_SMD:R_0402_1005Metric" V 12230 5075 50  0001 C CNN
@@
 3V3
 $Comp
-L power:GND #PWR0122
+L power:GND #PWR0603
 U 1 1 5E9441DB
 P 9825 6025
-F 0 "#PWR0122" H 9825 5775 50  0001 C CNN
+F 0 "#PWR0603" H 9825 5775 50  0001 C CNN
 F 1 "GND" H 9830 5852 50  0000 C CNN
 F 2 "" H 9825 6025 50  0001 C CNN
@@
 V_ALT
 $Comp
-L power:PWR_FLAG #FLG0104
+L power:PWR_FLAG #FLG0601
 U 1 1 5E9CDAED
 P 7100 4975
-F 0 "#FLG0104" H 7100 5050 50  0001 C CNN
+F 0 "#FLG0601" H 7100 5050 50  0001 C CNN
 F 1 "PWR_FLAG" H 7100 5125 50  0000 C CNN
 F 2 "" H 7100 4975 50  0001 C CNN

Commit message: Updated BOM for ordering parts
Parts:
- R601, R603: value R -> 100K; Link1 (none) -> https://www.digikey.com/product-detail/en/yageo/RC0402JR-07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; MPN1 (none) -> RC0402JR-07100KL; Short Description (none) -> RES SMD 100K OHM 5% 1/16W 0402; Standard Price (none) -> $0.00139
- R602: value R -> 453K; Link1 (none) -> https://www.digikey.com/product-detail/en/stackpole-electro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; MPN1 (none) -> RMCF0402FT453K; Short Description (none) -> RES 453K OHM 1% 1/16W 0402; Standard Price (none) -> 0.00149; Vendor1 Yageo -> Stackpole Electronics Inc
- U601: value TPS62821DLC -> TPS62821
Other:
- moved on the sheet: C603, R602, R603
Changed lines of the file:
@@
 P 8025 5325
 F 0 "U601" H 8000 5990 50  0000 C CNN
-F 1 "TPS62821DLC" H 8000 5899 50  0000 C CNN
+F 1 "TPS62821" H 8000 5899 50  0000 C CNN
 F 2 "leash:TPS62821DLC" H 7925 5275 50  0001 C CNN
 F 3 "http://www.ti.com/lit/ds/symlink/tps62823.pdf" H 7925 5275 50  0001 C CNN
@@
 P 7200 5475
 F 0 "R601" V 6993 5475 50  0000 C CNN
-F 1 "R" V 7084 5475 50  0000 C CNN
+F 1 "100K" V 7084 5475 50  0000 C CNN
 F 2 "Resistor_SMD:R_0402_1005Metric" V 7130 5475 50  0001 C CNN
 F 3 "~" H 7200 5475 50  0001 C CNN
 F 4 "-A1,-P" H 7200 5475 50  0001 C CNN "Population"
 F 5 "" H 7200 5475 50  0001 C CNN "Description"
-F 6 "" H 7200 5475 50  0001 C CNN "Link1"
-F 7 "" H 7200 5475 50  0001 C CNN "MPN1"
-F 8 "" H 7200 5475 50  0001 C CNN "Standard Price"
-F 9 "Yageo" H 7200 5475 50  0001 C CNN "Vendor1"
+F 6 "Yageo" H 7200 5475 50  0001 C CNN "Vendor1"
+F 7 "https://www.digikey.com/product-detail/en/yageo/RC0402JR-07100KL/311-100KJRCT-ND/729363" H 7200 5475 50  0001 C CNN "Link1"
+F 8 "RC0402JR-07100KL" H 7200 5475 50  0001 C CNN "MPN1"
+F 9 "RES SMD 100K OHM 5% 1/16W 0402" H 7200 5475 50  0001 C CNN "Short Description"
+F 10 "$0.00139" H 7200 5475 50  0001 C CNN "Standard Price"
 	1    7200 5475
 	0    1    1    0
@@
 L Device:R R602
 U 1 1 5D1DA985
-P 9825 5275
-F 0 "R602" H 9755 5229 50  0000 R CNN
-F 1 "R" H 9755 5320 50  0000 R CNN
-F 2 "Resistor_SMD:R_0402_1005Metric" V 9755 5275 50  0001 C CNN
-F 3 "~" H 9825 5275 50  0001 C CNN
-F 4 "-A1,-P" H 9825 5275 50  0001 C CNN "Population"
-F 5 "" H 9825 5275 50  0001 C CNN "Description"
-F 6 "" H 9825 5275 50  0001 C CNN "Link1"
-F 7 "" H 9825 5275 50  0001 C CNN "MPN1"
-F 8 "" H 9825 5275 50  0001 C CNN "Standard Price"
-F 9 "Yageo" H 9825 5275 50  0001 C CNN "Vendor1"
-	1    9825 5275
+P 10075 5275
+F 0 "R602" H 10005 5229 50  0000 R CNN
+F 1 "453K" H 10005 5320 50  0000 R CNN
+F 2 "Resistor_SMD:R_0402_1005Metric" V 10005 5275 50  0001 C CNN
+F 3 "~" H 10075 5275 50  0001 C CNN
+F 4 "-A1,-P" H 10075 5275 50  0001 C CNN "Population"
+F 5 "" H 10075 5275 50  0001 C CNN "Description"
+F 6 "Stackpole Electronics Inc" H 10075 5275 50  0001 C CNN "Vendor1"
+F 7 "https://www.digikey.com/product-detail/en/stackpole-electronics-inc/RMCF0402FT453K/RMCF0402FT453KTR-ND/1714738" H 10075 5275 50  0001 C CNN "Link1"
+F 8 "RMCF0402FT453K" H 10075 5275 50  0001 C CNN "MPN1"
+F 9 "RES 453K OHM 1% 1/16W 0402" H 10075 5275 50  0001 C CNN "Short Description"
+F 10 "0.00149" H 10075 5275 50  0001 C CNN "Standard Price"
+	1    10075 5275
 	-1   0    0    1
 $EndComp
@@
 L Device:R R603
 U 1 1 5D1DAF59
-P 9825 5675
-F 0 "R603" H 9755 5629 50  0000 R CNN
-F 1 "R" H 9755 5720 50  0000 R CNN
-F 2 "Resistor_SMD:R_0402_1005Metric" V 9755 5675 50  0001 C CNN
-F 3 "~" H 9825 5675 50  0001 C CNN
-F 4 "-A1,-P" H 9825 5675 50  0001 C CNN "Population"
-F 5 "" H 9825 5675 50  0001 C CNN "Description"
-F 6 "" H 9825 5675 50  0001 C CNN "Link1"
-F 7 "" H 9825 5675 50  0001 C CNN "MPN1"
-F 8 "" H 9825 5675 50  0001 C CNN "Standard Price"
-F 9 "Yageo" H 9825 5675 50  0001 C CNN "Vendor1"
-	1    9825 5675
+P 10075 5675
+F 0 "R603" H 10005 5629 50  0000 R CNN
+F 1 "100K" H 10005 5720 50  0000 R CNN
+F 2 "Resistor_SMD:R_0402_1005Metric" V 10005 5675 50  0001 C CNN
+F 3 "~" H 10075 5675 50  0001 C CNN
+F 4 "-A1,-P" H 10075 5675 50  0001 C CNN "Population"
+F 5 "" H 10075 5675 50  0001 C CNN "Description"
+F 6 "Yageo" H 10075 5675 50  0001 C CNN "Vendor1"
+F 7 "https://www.digikey.com/product-detail/en/yageo/RC0402JR-07100KL/311-100KJRCT-ND/729363" H 10075 5675 50  0001 C CNN "Link1"
+F 8 "RC0402JR-07100KL" H 10075 5675 50  0001 C CNN "MPN1"
+F 9 "RES SMD 100K OHM 5% 1/16W 0402" H 10075 5675 50  0001 C CNN "Short Description"
+F 10 "$0.00139" H 10075 5675 50  0001 C CNN "Standard Price"
+	1    10075 5675
 	-1   0    0    1
 $EndComp
@@
 $EndComp
 Wire Wire Line
-	9825 5125 9825 5075
-Wire Wire Line
-	9825 5075 9525 5075
+	10075 5125 10075 5075
+Wire Wire Line
+	10075 5075 9525 5075
 Wire Wire Line
 	9525 5125 9525 5075
@@
 	9525 5075 9300 5075
 Wire Wire Line
-	9825 5425 9825 5475
-Wire Wire Line
-	9825 5825 9825 5950
-Wire Wire Line
-	9825 5475 9525 5475
+	10075 5425 10075 5475
+Wire Wire Line
+	10075 5825 10075 5950
+Wire Wire Line
+	10075 5475 9525 5475
 Wire Wire Line
 	8650 5475 8650 5325
 Wire Wire Line
 	8650 5325 8425 5325
-Connection ~ 9825 5475
-Wire Wire Line
-	9825 5475 9825 5525
+Connection ~ 10075 5475
+Wire Wire Line
+	10075 5475 10075 5525
 Wire Wire Line
 	8425 5075 8800 5075
@@
 L Device:C C603
 U 1 1 5D20CB94
-P 10350 5575
-F 0 "C603" H 10465 5621 50  0000 L CNN
-F 1 "10 uF" H 10465 5530 50  0000 L CNN
-F 2 "Capacitor_SMD:C_0603_1608Metric" H 10388 5425 50  0001 C CNN
-F 3 "~" H 10350 5575 50  0001 C CNN
-F 4 "-A1,-P" H 10350 5575 50  0001 C CNN "Population"
-F 5 "CAP CER 10UF 6.3V X5R 0603" H 10350 5575 50  0001 C CNN "Description"
-F 6 "https://www.digikey.com/product-detail/en/samsung-electro-mechanics/CL10A106MQ8NNNC/1276-1119-1-ND/3889205" H 10350 5575 50  0001 C CNN "Link1"
-F 7 "CL10A106MQ8NNNC" H 10350 5575 50  0001 C CNN "MPN1"
-F 8 "$0.02215" H 10350 5575 50  0001 C CNN "Standard Price"
-F 9 "CAP CER 10UF 6.3V X5R 0603" H 10350 5575 50  0001 C CNN "Short Description"
-	1    10350 5575
-	1    0    0    -1
-$EndComp
-Wire Wire Line
-	10350 5425 10350 5075
-Connection ~ 9825 5075
-Wire Wire Line
-	10350 5725 10350 5950
-Wire Wire Line
-	10350 5950 9825 5950
-Connection ~ 9825 5950
-Wire Wire Line
-	9825 5950 9825 6025
+P 10600 5575
+F 0 "C603" H 10715 5621 50  0000 L CNN
+F 1 "10 uF" H 10715 5530 50  0000 L CNN
+F 2 "Capacitor_SMD:C_0603_1608Metric" H 10638 5425 50  0001 C CNN
+F 3 "~" H 10600 5575 50  0001 C CNN
+F 4 "-A1,-P" H 10600 5575 50  0001 C CNN "Population"
+F 5 "CAP CER 10UF 6.3V X5R 0603" H 10600 5575 50  0001 C CNN "Description"
+F 6 "https://www.digikey.com/product-detail/en/samsung-electro-mechanics/CL10A106MQ8NNNC/1276-1119-1-ND/3889205" H 10600 5575 50  0001 C CNN "Link1"
+F 7 "CL10A106MQ8NNNC" H 10600 5575 50  0001 C CNN "MPN1"
+F 8 "$0.02215" H 10600 5575 50  0001 C CNN "Standard Price"
+F 9 "CAP CER 10UF 6.3V X5R 0603" H 10600 5575 50  0001 C CNN "Short Description"
+	1    10600 5575
+	1    0    0    -1
+$EndComp
+Wire Wire Line
+	10600 5425 10600 5075
+Connection ~ 10075 5075
+Wire Wire Line
+	10600 5725 10600 5950
+Wire Wire Line
+	10600 5950 10075 5950
+Connection ~ 10075 5950
+Wire Wire Line
+	10075 5950 10075 6025
 $Comp
 L Device:C C601
@@
 3V3_BUCK_VOUT
 Wire Wire Line
-	9825 5075 10350 5075
-Connection ~ 10350 5075
-Wire Wire Line
-	10350 5075 12150 5075
+	10075 5075 10600 5075
+Connection ~ 10600 5075
+Wire Wire Line
+	10600 5075 12150 5075
 $Comp
 L Device:R R604
@@
 L power:GND #PWR0603
 U 1 1 5E9441DB
-P 9825 6025
-F 0 "#PWR0603" H 9825 5775 50  0001 C CNN
-F 1 "GND" H 9830 5852 50  0000 C CNN
-F 2 "" H 9825 6025 50  0001 C CNN
-F 3 "" H 9825 6025 50  0001 C CNN
-	1    9825 6025
-	1    0    0    -1
-$EndComp
+P 10075 6025
+F 0 "#PWR0603" H 10075 5775 50  0001 C CNN
+F 1 "GND" H 10080 5852 50  0000 C CNN
+F 2 "" H 10075 6025 50  0001 C CNN
+F 3 "" H 10075 6025 50  0001 C CNN
+	1    10075 6025
+	1    0    0    -1
+$EndComp

Commit message: Updated after latest Rev B build and BOM update, including new STEP file export
Parts:
- C601, C602, C603, R601, R602, R603, R604, U601: Population -A1,-P -> (none)
- L601: value INDUCTOR -> 0.47U; MPN1 (none) -> ASMPM-0806-R47M-T; Population -A1,-P -> (none)
Changed lines of the file:
@@
 F 2 "leash:TPS62821DLC" H 7925 5275 50  0001 C CNN
 F 3 "http://www.ti.com/lit/ds/symlink/tps62823.pdf" H 7925 5275 50  0001 C CNN
-F 4 "-A1,-P" H 8025 5325 50  0001 C CNN "Population"
+F 4 "" H 8025 5325 50  0001 C CNN "Population"
 F 5 "IC REG BUCK ADJ 1A 8VSON-HR" H 8025 5325 50  0001 C CNN "Description"
 F 6 "https://www.digikey.com/product-detail/en/texas-instruments/TPS62821DLCR/296-50127-1-ND/9462910" H 8025 5325 50  0001 C CNN "Link1"
@@
 F 2 "Resistor_SMD:R_0402_1005Metric" V 7130 5475 50  0001 C CNN
 F 3 "~" H 7200 5475 50  0001 C CNN
-F 4 "-A1,-P" H 7200 5475 50  0001 C CNN "Population"
+F 4 "" H 7200 5475 50  0001 C CNN "Population"
 F 5 "" H 7200 5475 50  0001 C CNN "Description"
 F 6 "Yageo" H 7200 5475 50  0001 C CNN "Vendor1"
@@
 P 9050 5075
 F 0 "L601" H 9050 5290 50  0000 C CNN
-F 1 "INDUCTOR" H 9050 5199 50  0000 C CNN
+F 1 "0.47U" H 9050 5199 50  0000 C CNN
 F 2 "leash:L_0806_2012Metric" H 9050 5075 50  0001 C CNN
 F 3 "~" H 9050 5075 50  0001 C CNN
-F 4 "-A1,-P" H 9050 5075 50  0001 C CNN "Population"
+F 4 "" H 9050 5075 50  0001 C CNN "Population"
+F 5 "ASMPM-0806-R47M-T" H 9050 5075 50  0001 C CNN "MPN1"
 	1    9050 5075
 	1    0    0    -1
@@
 F 2 "Resistor_SMD:R_0402_1005Metric" V 10005 5275 50  0001 C CNN
 F 3 "~" H 10075 5275 50  0001 C CNN
-F 4 "-A1,-P" H 10075 5275 50  0001 C CNN "Population"
+F 4 "" H 10075 5275 50  0001 C CNN "Population"
 F 5 "" H 10075 5275 50  0001 C CNN "Description"
 F 6 "Stackpole Electronics Inc" H 10075 5275 50  0001 C CNN "Vendor1"
@@
 F 2 "Resistor_SMD:R_0402_1005Metric" V 10005 5675 50  0001 C CNN
 F 3 "~" H 10075 5675 50  0001 C CNN
-F 4 "-A1,-P" H 10075 5675 50  0001 C CNN "Population"
+F 4 "" H 10075 5675 50  0001 C CNN "Population"
 F 5 "" H 10075 5675 50  0001 C CNN "Description"
 F 6 "Yageo" H 10075 5675 50  0001 C CNN "Vendor1"
@@
 F 2 "Capacitor_SMD:C_0402_1005Metric" H 9563 5125 50  0001 C CNN
 F 3 "~" H 9525 5275 50  0001 C CNN
-F 4 "-A1,-P" H 9525 5275 50  0001 C CNN "Population"
+F 4 "" H 9525 5275 50  0001 C CNN "Population"
 F 5 "CAP CER 100PF 50V C0G/NPO 0402" H 9525 5275 50  0001 C CNN "Description"
 F 6 "https://www.digikey.com/product-detail/en/yageo/CC0402JRNPO9BN101/311-1024-1-ND/302941" H 9525 5275 50  0001 C CNN "Link1"
@@
 F 2 "Capacitor_SMD:C_0603_1608Metric" H 10638 5425 50  0001 C CNN
 F 3 "~" H 10600 5575 50  0001 C CNN
-F 4 "-A1,-P" H 10600 5575 50  0001 C CNN "Population"
+F 4 "" H 10600 5575 50  0001 C CNN "Population"
 F 5 "CAP CER 10UF 6.3V X5R 0603" H 10600 5575 50  0001 C CNN "Description"
 F 6 "https://www.digikey.com/product-detail/en/samsung-electro-mechanics/CL10A106MQ8NNNC/1276-1119-1-ND/3889205" H 10600 5575 50  0001 C CNN "Link1"
@@
 F 2 "Capacitor_SMD:C_0402_1005Metric" H 6313 5175 50  0001 C CNN
 F 3 "~" H 6275 5325 50  0001 C CNN
-F 4 "-A1,-P" H 6275 5325 50  0001 C CNN "Population"
+F 4 "" H 6275 5325 50  0001 C CNN "Population"
 F 5 "CAP CER 0.1UF 10V X5R 0402" H 6275 5325 50  0001 C CNN "Description"
 F 6 "https://www.digikey.com/product-detail/en/samsung-electro-mechanics/CL05A104MP5NNNC/1276-1443-1-ND/3889529" H 6275 5325 50  0001 C CNN "Link1"
@@
 F 2 "Resistor_SMD:R_0402_1005Metric" V 12230 5075 50  0001 C CNN
 F 3 "~" H 12300 5075 50  0001 C CNN
-F 4 "-A1,-P" H 12370 4984 50  0001 L CNN "Population"
+F 4 "" H 12370 4984 50  0001 L CNN "Population"
 F 5 "RES 0 OHM JUMPER 1/16W 0402" H 12300 5075 50  0001 C CNN "Description"
 F 6 "https://www.digikey.com/product-detail/en/stackpole-electronics-inc/RMCF0402ZT0R00/RMCF0402ZT0R00TR-ND/1756905" H 12300 5075 50  0001 C CNN "Link1"

Commit message: Revisions and fixes for Rev B board in preparation for Rev C start. Changed how we handle the MSP430 and how it connects to the cc1352r. Also some part swaps and pin swaps on the cc1352r. Fixes #4 and #5.
Parts:
- removed R604: 0, Resistor_SMD:R_0402_1005Metric, symbol Device:R
- added F601: Polyfuse, Resistor_SMD:R_0603_1608Metric, symbol Device:Polyfuse
- C601: value 1 uF -> 1U
- C602: value 100 pF -> 100P
- C603: value 10 uF -> 10U
Changed lines of the file:
@@
 P 9525 5275
 F 0 "C602" H 9640 5321 50  0000 L CNN
-F 1 "100 pF" H 9640 5230 50  0000 L CNN
+F 1 "100P" H 9640 5230 50  0000 L CNN
 F 2 "Capacitor_SMD:C_0402_1005Metric" H 9563 5125 50  0001 C CNN
 F 3 "~" H 9525 5275 50  0001 C CNN
@@
 P 10600 5575
 F 0 "C603" H 10715 5621 50  0000 L CNN
-F 1 "10 uF" H 10715 5530 50  0000 L CNN
+F 1 "10U" H 10715 5530 50  0000 L CNN
 F 2 "Capacitor_SMD:C_0603_1608Metric" H 10638 5425 50  0001 C CNN
 F 3 "~" H 10600 5575 50  0001 C CNN
@@
 P 6275 5325
 F 0 "C601" H 6390 5371 50  0000 L CNN
-F 1 "1 uF" H 6390 5280 50  0000 L CNN
+F 1 "1U" H 6390 5280 50  0000 L CNN
 F 2 "Capacitor_SMD:C_0402_1005Metric" H 6313 5175 50  0001 C CNN
 F 3 "~" H 6275 5325 50  0001 C CNN
@@
 Wire Wire Line
 	10600 5075 12150 5075
-$Comp
-L Device:R R604
-U 1 1 5E38DA29
-P 12300 5075
-F 0 "R604" H 12370 5166 50  0000 L CNN
-F 1 "0" H 12370 5075 50  0000 L CNN
-F 2 "Resistor_SMD:R_0402_1005Metric" V 12230 5075 50  0001 C CNN
-F 3 "~" H 12300 5075 50  0001 C CNN
-F 4 "" H 12370 4984 50  0001 L CNN "Population"
-F 5 "RES 0 OHM JUMPER 1/16W 0402" H 12300 5075 50  0001 C CNN "Description"
-F 6 "https://www.digikey.com/product-detail/en/stackpole-electronics-inc/RMCF0402ZT0R00/RMCF0402ZT0R00TR-ND/1756905" H 12300 5075 50  0001 C CNN "Link1"
-F 7 "RMCF0402ZT0R00" H 12300 5075 50  0001 C CNN "MPN1"
-F 8 "$0.00127" H 12300 5075 50  0001 C CNN "Standard Price"
-F 9 "Stackpole Electronics Inc" H 12300 5075 50  0001 C CNN "Vendor1"
-F 10 "RES 0 OHM JUMPER 1/16W 0402" H 12300 5075 50  0001 C CNN "Short Description"
-	1    12300 5075
-	0    1    1    0
-$EndComp
 Text Label 5575 5075 0    79   ~ 0
 3V3_BUCK_IN
@@
 Wire Wire Line
 	7100 5075 7450 5075
+$Comp
+L Device:Polyfuse F?
+U 1 1 5F2F707F
+P 12300 5075
+AR Path="/5D062750/5F2F707F" Ref="F?"  Part="1"
+AR Path="/5D0620A4/5F2F707F" Ref="F601"  Part="1"
+F 0 "F601" V 12200 5075 50  0000 C CNN
+F 1 "Polyfuse" V 12400 5075 50  0000 C CNN
+F 2 "Resistor_SMD:R_0603_1608Metric" H 12350 4875 50  0001 L CNN
+F 3 "~" H 12300 5075 50  0001 C CNN
+F 4 "https://www.digikey.com/product-detail/en/yageo/RC0603JR-070RL/311-0-0GRTR-ND/726675" H 12300 5075 50  0001 C CNN "Link1"
+F 5 "RC0603JR-070RL" H 12300 5075 50  0001 C CNN "MPN1"
+F 6 "RES SMD 0 OHM JUMPER 1/10W 0603" H 12300 5075 50  0001 C CNN "Short Description"
+F 7 "0.00196" H 12300 5075 50  0001 C CNN "Standard Price"
+F 8 "Yageo" H 12300 5075 50  0001 C CNN "Vendor1"
+	1    12300 5075
+	0    1    1    0
+$EndComp
 $EndSCHEMATC
