File: hw/LeashPCB/Boost.sch (KiCad schematic (older format))
At the start: 9 parts, among them U601 TPS62821

Commit message: Updating some of the standard pricing on the schematic
Parts:
- R601, R603: Standard Price $0.00139 -> 0.00139
Changed lines of the file:
@@
 F 8 "RC0402JR-07100KL" H 7200 5475 50  0001 C CNN "MPN1"
 F 9 "RES SMD 100K OHM 5% 1/16W 0402" H 7200 5475 50  0001 C CNN "Short Description"
-F 10 "$0.00139" H 7200 5475 50  0001 C CNN "Standard Price"
+F 10 "0.00139" H 7200 5475 50  0001 C CNN "Standard Price"
 	1    7200 5475
 	0    1    1    0
@@
 F 8 "RC0402JR-07100KL" H 10075 5675 50  0001 C CNN "MPN1"
 F 9 "RES SMD 100K OHM 5% 1/16W 0402" H 10075 5675 50  0001 C CNN "Short Description"
-F 10 "$0.00139" H 10075 5675 50  0001 C CNN "Standard Price"
+F 10 "0.00139" H 10075 5675 50  0001 C CNN "Standard Price"
 	1    10075 5675
 	-1   0    0    1
