File: hw/Freedom/BeagleConnect Freedom.kicad_pcb (KiCad board)
At the start: 4 copper layers, 41.2 x 33.3 mm, 156 parts, among them J1 Conn_01x02_Male, J2 TAG-CONNECT-10, J3 TAG-CONNECT-10, J4 mikroBUS, J5 mikroBUS, J6 UFL, J7 UFL, J8 UFL, P1 USB_C_Receptacle_USB2.0, Q1 CJ2305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

Commit message: HW: Freedom: rev C2 (1103)
* Rotate mikroBUS to avoid buttons https://github.com/jadonk/beagleconnect/issues/29
* Released to prototype
Parts:
- turned J5 to 270 degrees
Routing:
- net MOSI: track 31.0 -> 55.7 mm, vias 3 -> 4
- net MISO: track 22.9 -> 44.1 mm, vias 2 -> 3
- net SCK: track 27.1 -> 37.4 mm, vias 2 -> 3
- net INT_MB2: track 19.0 -> 29.2 mm
- net SCL: track 72.6 -> 82.2 mm
- net PWM_MB2: track 20.9 -> 30.4 mm
- net 5V: track 63.4 -> 71.9 mm, vias 4 -> 5
- net SDA: track 70.1 -> 77.0 mm, vias 4 -> 6
- net CS_MB2: track 17.9 -> 12.0 mm
- net USER_BOOT: track 65.3 -> 71.1 mm, vias 4 -> 5
- net CC1352_TX_MB2_RX: track 21.7 -> 26.6 mm, vias 1 -> 4
- net AN_MB2: track 21.3 -> 24.6 mm
- net INT_SENSOR: track 66.9 -> 69.9 mm
- net CC1352_RX_MB2_TX: track 25.1 -> 28.1 mm, vias 2 -> 4
- net LED2: track 26.1 -> 23.7 mm
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
Commit message: From Fiona
Parts:
- removed R29: 0, Resistor_SMD:R_0402_1005Metric
- C28: value 100N -> DNP
- C31: value DNP -> 0.5pF
- C34: value 12P -> 0R
- C35, C36: value 100N -> 0R
- C37: value 1P -> 1nF
- L5: value 0 -> 2.0pF
- R51: moved to B.Cu
- moved R51 5.02 mm to (34.2, -31.0), turned to 0 degrees
- moved C13 3.22 mm to (28.6, -27.1)
- moved R34 3.21 mm to (27.6, -27.1)
- moved R35 3.06 mm to (29.8, -27.1)
- moved C41 3.00 mm to (28.6, -29.2), turned to 180 degrees
- moved C12 2.36 mm to (32.8, -28.1), turned to 270 degrees
- moved R14 1.66 mm to (28.8, -25.1)
- moved R13 1.64 mm to (29.8, -25.2)
- moved U3 1.34 mm to (30.9, -27.7)
- moved D12 0.87 mm to (34.3, -30.0), turned to 0 degrees
- moved C45 0.42 mm to (28.6, -28.0)
- moved C14 0.37 mm to (28.6, -26.9)
- moved L2 0.17 mm to (29.2, -25.4)
- moved R28 0.07 mm to (23.8, -22.9)
- moved P1 0.06 mm to (37.5, -20.9)
Connections:
- B2 pad 2: GND -> /RF/VDDR
- U1 pad 30: Net-(R29-Pad2) -> SDA
- U1 pad 31: Net-(U1-Pad31) -> SCL
Routing:
- net SCL: track 82.2 -> 98.0 mm, vias 3 -> 4
- net /RF/VDDR: track 30.3 -> 41.2 mm, vias 3 -> 4
- net GND: track 160.6 -> 169.5 mm, vias 142 -> 135
- net SDA: track 77.0 -> 82.9 mm, vias 6 -> 8
- net 3V3: track 205.8 -> 210.4 mm
- net Net-(R51-Pad1): track 4.02 -> 8.00 mm, vias 1 -> 2
- net Net-(R28-Pad2): track 3.61 -> 1.29 mm
- net V_ALT: track 30.7 -> 28.4 mm, vias 4 -> 3
- net INT_HDC2010: track 1.80 -> 3.81 mm
- net Net-(R29-Pad2): track 1.91 -> 0.00 mm, vias 1 -> 0
- net /USB Input/MSP_PUR: track 8.35 -> 6.68 mm
- net Net-(L2-Pad1): track 3.39 -> 2.06 mm
- net BUZZER_CTL: track 13.6 -> 14.6 mm
- net INT_SENSOR: track 69.9 -> 70.9 mm
- net CC1352_RX_MSP430_TX: track 32.6 -> 33.4 mm
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Other:
- board size 41.2 x 33.3 mm -> 41.3 x 33.4 mm
- board text added: "BOOT"
- board text added: "CC1352P BeagleConnect Freedom Rev C3"
- board text added: "RESET"
- board text removed: "CC1352P BeagleConnect Freedom Rev C2"
