File: hw/Freedom_C4/BeagleConnect Freedom.kicad_pcb (KiCad board)
At the start: 4 copper layers, 1262.4 x 74.9 mm, 175 parts, among them J1 Conn_01x02_Female, J2 TAG-CONNECT-10, J3 TAG-CONNECT-10, J4 mikroBUS, J5 mikroBUS, J8 UFL, P1 USB_C_Receptacle_USB2.0, Q1 CJ2305, Q2 2N7002PW, Q3 BC856S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

Commit message: Update to version C5
Parts:
- added SH1: Shield, leash:SHIELDING_27.5x15.5x0.2mm, B.Cu at (275.0, 44.2)
- C48: value 12P -> 7P
- D9: value BAT54 -> PMEG6020ER,115
- F1: value 500mA -> 3A
- J1: value Conn_01x02_Female -> ST-FH-254-0144-02
- moved C54 3.97 mm to (273.8, 48.4), turned to 0 degrees
- moved B1 3.43 mm to (276.7, 49.2)
- moved C11 3.03 mm to (277.2, 40.4), turned to 90 degrees
- moved C24 2.66 mm to (283.6, 49.9), turned to 270 degrees
- moved L8 1.55 mm to (276.4, 40.1), turned to 270 degrees
- moved L10 1.28 mm to (276.5, 45.8), turned to 315 degrees
- moved L3 1.26 mm to (284.9, 41.3), turned to 180 degrees
- moved C14 1.20 mm to (285.8, 36.2)
- moved L12 1.18 mm to (274.4, 44.2)
- moved C46 1.17 mm to (274.8, 43.1)
- moved C20 1.17 mm to (279.2, 40.9)
- moved R33 1.17 mm to (280.2, 40.9)
- moved R36 1.17 mm to (284.4, 39.7)
- moved R39 1.17 mm to (283.3, 40.9)
- moved C15 1.17 mm to (277.7, 47.1)
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- renumbered P1 to USB1
Connections:
- C53 pad 1: Net-(C52-Pad2) -> Net-(C53-Pad1)
- C53 pad 2: Net-(C53-Pad2) -> Net-(C52-Pad2)
- L15 pad 2: Net-(B1-Pad1) -> Net-(C29-Pad2)
- R51 pad 2: GND -> 3V3
- U11 pad 4: Net-(C53-Pad2) -> Net-(C53-Pad1)
- U4 pad 14: /RF/~FLASH_CS -> ~FLASH_CS
Routing:
- net GND: track 170.5 -> 215.0 mm, vias 214 -> 224
- net ~FLASH_CS: track 14.0 -> 47.0 mm, vias 1 -> 2
- net VDDS: track 71.5 -> 47.8 mm
- net 2.4G: track 68.0 -> 59.7 mm
- net USER_BOOT: track 63.1 -> 55.3 mm
- net 3V3: track 81.5 -> 74.4 mm, vias 20 -> 19
- net LED1: track 39.1 -> 32.2 mm
- net RF_SW_CTRL1: track 43.2 -> 37.6 mm
- net ~CHG: track 11.5 -> 15.8 mm, vias 0 -> 2
- net Net-(C53-Pad2): track 4.20 -> 0.00 mm
- net /RF/RF_SUB_1GHZ_P: track 5.78 -> 1.92 mm
- net /RF/RF_SUB_1GHZ_N: track 5.78 -> 1.92 mm
- net /RF/RF_2_4GHZ_P: track 5.78 -> 1.92 mm
- net /RF/RF_2_4GHZ_N: track 5.78 -> 1.92 mm
- net 5V: track 97.8 -> 94.4 mm
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- added copper zone on F.Cu, net VDDS
Other:
- outline, holes or cut-outs redrawn
- board text added: "3V3"
- board text added: "5V"
- board text added: "BZ1"
- board text added: "GND"
- board text added: "P1"
- board text added: "P2"
- board text added: "P3"
- board text added: "P4"
- board text added: "Rev C5"
- board text added: "SH1"
- board text added: "U6"
- board text removed: "Rev C4"
